File: FPGA-BOARDver3/POWER_REGULATION2.kicad_sch (KiCad schematic)
At the start: 63 parts, among them J7 Conn_01x06_Pin, Q8 FDV301N, U22 TPS65400RGZT, U4 NC7WZ07P6X

Commit message: All pages complete , pi header left
Parts:
- removed S1: PTS645SK50SMTR92LFS, footprints:SW_PTS645SK50SMTR92LFS, symbol PTS645SK50SMTR92LFS:PTS645SK50SMTR92LFS
- removed U4: NC7WZ07P6X, footprints:NC7WZ07P6X, symbol NC7WZ07P6X:NC7WZ07P6X
- added S1: PTS645SK50SMTR92LFS, footprints:SW_PTS645SK50SMTR92LFS, symbol PTS645SK50SMTR92LFS_:PTS645SK50SMTR92LFS
- added U9: NC7WZ07P6X, footprints:NC7WZ07P6X, symbol NC7WZ07P6X:NC7WZ07P6X
Connections:
- net GNDREF: now also S1.3
- net PG_ALL: now also U9.3 (A2)
- net PS_POR_B: now also S1.1, U9.4 (Y2)
- new net VCC: U9.5 (VCC)
Changed lines of the file:
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@@
 	(wire
 		(pts
-			(xy 85.09 152.4) (xy 95.25 152.4)
+			(xy 85.09 152.4) (xy 96.52 152.4)
 		)
 		(stroke
@@
 	)
 	(symbol
-		(lib_id "NC7WZ07P6X:NC7WZ07P6X")
-		(at 99.06 147.32 0)
-		(unit 1)
-		(exclude_from_sim no)
-		(in_bom yes)
-		(on_board yes)
-		(dnp no)
-		(property "Reference" "U4"
-			(at 99.314 145.796 0)
-			(effects
-				(font
-					(size 1.27 1.27)
-				)
-			)
-		)
-		(property "Value" "NC7WZ07P6X"
-			(at 99.06 147.32 0)
-			(effects
-				(font
-					(size 1.27 1.27)
-				)
-			)
-		)
-		(property "Footprint" "footprints:NC7WZ07P6X"
-			(at 99.06 147.32 0)
-			(effects
-				(font
-					(size 1.27 1.27)
-				)
-				(justify bottom)
-				(hide yes)
-			)
-		)
-		(property "Datasheet" ""
-			(at 99.06 147.32 0)
-			(effects
-				(font
-					(size 1.27 1.27)
-				)
-				(hide yes)
-			)
-		)
-		(property "Description" ""
-			(at 99.06 147.32 0)
-			(effects
-				(font
-					(size 1.27 1.27)
-				)
-				(hide yes)
-			)
-		)
-		(property "SUPPLIER" "FAIRCHILD SEMICONDUCTOR"
-			(at 99.06 147.32 0)
-			(effects
-				(font
-					(size 1.27 1.27)
-				)
-				(justify bottom)
-				(hide yes)
-			)
-		)
-		(property "OC_FARNELL" "1470998"
-			(at 99.06 147.32 0)
-			(effects
-				(font
-					(size 1.27 1.27)
-				)
-				(justify bottom)
-				(hide yes)
-			)
-		)
-		(property "OC_NEWARK" "58K9469"
-			(at 99.06 147.32 0)
-			(effects
-				(font
-					(size 1.27 1.27)
-				)
-				(justify bottom)
-				(hide yes)
-			)
-		)
-		(property "MPN" "NC7WZ07P6X"
-			(at 99.06 147.32 0)
-			(effects
-				(font
-					(size 1.27 1.27)
-				)
-				(justify bottom)
-				(hide yes)
-			)
-		)
-		(property "PACKAGE" "SC-70-6"
-			(at 99.06 147.32 0)
-			(effects
-				(font
-					(size 1.27 1.27)
-				)
-				(justify bottom)
-				(hide yes)
-			)
-		)
-		(pin "3"
-		)
-		(pin "4"
-		)
-		(instances
-			(project "FPGA-BOARDver3"
-				(path "/4a327bdf-04e5-4836-9c0a-5fb801c23f64/96f87610-c13d-493b-977a-68dc2191f3d9"
-					(reference "U4")
-					(unit 1)
-				)
-			)
-		)
-	)
-	(symbol
 		(lib_id "power:+3V3")
 		(at 247.65 38.1 270)
@@
 	)
 	(symbol
-		(lib_id "PTS645SK50SMTR92LFS:PTS645SK50SMTR92LFS")
-		(at 120.65 168.91 0)
-		(unit 1)
-		(exclude_from_sim no)
-		(in_bom yes)
-		(on_board yes)
-		(dnp no)
-		(fields_autoplaced yes)
-		(property "Reference" "S1"
-			(at 121.92 167.6399 0)
-			(effects
-				(font
-					(size 1.27 1.27)
-				)
-				(justify left)
-			)
-		)
-		(property "Value" "PTS645SK50SMTR92LFS"
-			(at 121.92 170.1799 0)
-			(effects
-				(font
-					(size 1.27 1.27)
-				)
-				(justify left)
-			)
-		)
-		(property "Footprint" "footprints:SW_PTS645SK50SMTR92LFS"
-			(at 120.65 168.91 0)
-			(effects
-				(font
-					(size 1.27 1.27)
-				)
-				(justify bottom)
-				(hide yes)
-			)
-		)
-		(property "Datasheet" ""
-			(at 120.65 168.91 0)
-			(effects
-				(font
-					(size 1.27 1.27)
-				)
-				(hide yes)
-			)
-		)
-		(property "Description" ""
-			(at 120.65 168.91 0)
-			(effects
-				(font
-					(size 1.27 1.27)
-				)
-				(hide yes)
-			)
-		)
-		(property "STANDARD" "Manufacturer Recommendations"
-			(at 120.65 168.91 0)
-			(effects
-				(font
-					(size 1.27 1.27)
-				)
-				(justify bottom)
-				(hide yes)
-			)
-		)
-		(property "MANUFACTURER" "CnK"
-			(at 120.65 168.91 0)
-			(effects
-				(font
-					(size 1.27 1.27)
-				)
-				(justify bottom)
-				(hide yes)
-			)
-		)
-		(pin "1"
-		)
-		(pin "3"
-		)
-		(instances
-			(project ""
-				(path "/4a327bdf-04e5-4836-9c0a-5fb801c23f64/96f87610-c13d-493b-977a-68dc2191f3d9"
-					(reference "S1")
-					(unit 1)
-				)
-			)
-		)
-	)
-	(symbol
 		(lib_id "power:+3V3")
 		(at 247.65 64.77 270)
@@
 	)
 	(symbol
+		(lib_id "PTS645SK50SMTR92LFS_:PTS645SK50SMTR92LFS")
+		(at 120.65 168.91 0)
+		(unit 1)
+		(exclude_from_sim no)
+		(in_bom yes)
+		(on_board yes)
+		(dnp no)
+		(fields_autoplaced yes)
+		(property "Reference" "S1"
+			(at 121.92 167.6399 0)
+			(effects
+				(font
+					(size 1.27 1.27)
+				)
+				(justify left)
+			)
+		)
+		(property "Value" "PTS645SK50SMTR92LFS"
+			(at 121.92 170.1799 0)
+			(effects
+				(font
+					(size 1.27 1.27)
+				)
+				(justify left)
+			)
+		)
+		(property "Footprint" "footprints:SW_PTS645SK50SMTR92LFS"
+			(at 120.65 168.91 0)
+			(effects
+				(font
+					(size 1.27 1.27)
+				)
+				(justify bottom)
+				(hide yes)
+			)
+		)
+		(property "Datasheet" ""
+			(at 120.65 168.91 0)
+			(effects
+				(font
+					(size 1.27 1.27)
+				)
+				(hide yes)
+			)
+		)
+		(property "Description" ""
+			(at 120.65 168.91 0)
+			(effects
+				(font
+					(size 1.27 1.27)
+				)
+				(hide yes)
+			)
+		)
+		(property "STANDARD" "Manufacturer Recommendations"
+			(at 120.65 168.91 0)
+			(effects
+				(font
+					(size 1.27 1.27)
+				)
+				(justify bottom)
+				(hide yes)
+			)
+		)
+		(property "MANUFACTURER" "CnK"
+			(at 120.65 168.91 0)
+			(effects
+				(font
+					(size 1.27 1.27)
+				)
+				(justify bottom)
+				(hide yes)
+			)
+		)
+		(pin "4"
+		)
+		(pin "3"
+		)
+		(pin "1"
+		)
+		(pin "2"
+		)
+		(instances
+			(project "FPGA-BOARDver3"
+				(path "/4a327bdf-04e5-4836-9c0a-5fb801c23f64/96f87610-c13d-493b-977a-68dc2191f3d9"
+					(reference "S1")
+					(unit 1)
+				)
+			)
+		)
+	)
+	(symbol
 		(lib_id "power:GNDREF")
 		(at 247.65 127 90)
@@
 					(unit 1)
 				)
+			)
+		)
+	)
+	(symbol
+		(lib_name "NC7WZ07P6X_1")
+		(lib_id "NC7WZ07P6X:NC7WZ07P6X")
+		(at 102.87 152.4 0)
+		(unit 1)
+		(exclude_from_sim no)
+		(in_bom yes)
+		(on_board yes)
+		(dnp no)
+		(property "Reference" "U9"
+			(at 101.092 150.114 0)
+			(effects
+				(font
+					(size 1.27 1.27)
+				)
+			)
+		)
+		(property "Value" "NC7WZ07P6X"
+			(at 100.33 148.082 0)
+			(effects
+				(font
+					(size 1.27 1.27)
+				)
+			)
+		)
+		(property "Footprint" "footprints:NC7WZ07P6X"
+			(at 102.362 145.542 0)
+			(effects
+				(font
+					(size 1.27 1.27)
+				)
+				(justify bottom)
+				(hide yes)
+			)
+		)
+		(property "Datasheet" ""
+			(at 102.87 152.4 0)
+			(effects
+				(font
+					(size 1.27 1.27)
+				)
+				(hide yes)
+			)
+		)
+		(property "Description" ""
+			(at 102.87 152.4 0)
+			(effects
+				(font
+					(size 1.27 1.27)
+				)
+				(hide yes)
+			)
+		)
+		(property "SUPPLIER" "FAIRCHILD SEMICONDUCTOR"
+			(at 104.902 145.542 0)
+			(effects
+				(font
+					(size 1.27 1.27)
+				)
+				(justify bottom)
+				(hide yes)
+			)
+		)
+		(property "OC_FARNELL" "1470998"
+			(at 107.188 148.336 0)
+			(effects
+				(font
+					(size 1.27 1.27)
+				)
+				(justify bottom)
+				(hide yes)
+			)
+		)
+		(property "OC_NEWARK" "58K9469"
+			(at 105.918 149.098 0)
+			(effects
+				(font
+					(size 1.27 1.27)
+				)
+				(justify bottom)
+				(hide yes)
+			)
+		)
+		(property "MPN" "NC7WZ07P6X"
+			(at 102.87 146.304 0)
+			(effects
+				(font
+					(size 1.27 1.27)
+				)
+				(justify bottom)
+				(hide yes)
+			)
+		)
+		(property "PACKAGE" "SC-70-6"
+			(at 105.664 147.574 0)
+			(effects
+				(font
+					(size 1.27 1.27)
+				)
+				(justify bottom)
+				(hide yes)
+			)
+		)
+		(pin "6"
+		)
+		(pin "5"
+		)
+		(pin "1"
+		)
+		(pin "2"
+		)
+		(pin "3"
+		)
+		(pin "4"
+		)
+		(instances
+			(project ""
+				(path "/4a327bdf-04e5-4836-9c0a-5fb801c23f64/96f87610-c13d-493b-977a-68dc2191f3d9"
+					(reference "U9")
+					(unit 1)
+				)

Commit message: update
Parts:
- removed U9: NC7WZ07P6X, footprints:NC7WZ07P6X, symbol NC7WZ07P6X:NC7WZ07P6X
- added C171, C174, C175: 100nF, footprints:C_0402, symbol Device:C
- added C172, C81: 4.7uF, footprints:C_0402, symbol Device:C
- added C173: 1uF, footprints:C_0402, symbol Device:C
- added CR2: 1SS352, footprints:USC_TOS, symbol 1SS352:1SS352
- added R187: 15K, footprints:R_0402, symbol Device:R_US
- added R188: 310, footprints:R_0402, symbol Device:R_US
- added U19: NL17SZ17XV5T2G, footprints:SOT553-5_ONS, symbol NL17SZ17XV5T2G:NL17SZ17XV5T2G_Modified
- added U20: FPF1018, footprints:MLP6_2X2_ONS, symbol FPF1018:FPF1018
- added U21: NC7WZ07P6X, footprints:NC7WZ07P6X, symbol NC7WZ07P6X:NC7WZ07P6X_modified
- added U9: SIP32510DT-T1-GE3, footprints:SIP32510DT-T1-GE3_VIS, symbol SIP32510DT_T1_GE3:SIP32510DT-T1-GE3
- C33: value 4.7uF -> 100nF
- D25: footprint LED_SMD:LED_0402_1005Metric -> footprints:LED_0402_1005Metric
- R92: value 100k -> 15K
Connections:
- net +1V8: now also C172.1, C173.1, U20.2 (VIN), U20.3 (VIN), U9.5 (IN), U9.6 (IN)
- net +3.3V: now also C33.1, U19.5 (VCC)
- net GNDREF: now also C171.2, C172.2, C173.2, C174.2, C175.2, C81.2, R188.2, U19.3 (GND), U20.6 (GND), U20.7 (EPAD), U21.2 (GND), U9.4 (GND)
- net PG_ALL: now also CR2.1, R187.2, U20.1 (ON), U9.3 (EN); no longer C33.1, Q8.1
- net PS_POR_B: now also U21.4 (Y2)
- new net AVCC3V3: C175.1, U21.5 (VCC)
- new net PG_ALL_DLY: C81.1, CR2.2, R187.1, U19.2
- new net PG_ALL_EDGE: Q8.1, U19.4, U21.3 (A2)
- new net VCC1V8_IO: C171.1, C174.1, R188.1, U20.4 (VOUT), U20.5 (VOUT), U9.1 (OUT), U9.2 (OUT)
Other:
- moved on the sheet: C33, D25, J7, Q8, R111, R112, R113, R92, R93, R94, S1

Commit message: schematic pages for review
Changed lines of the file:
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@@
 	)
 	(symbol
+		(lib_name "NC7WZ07P6X_modified_1")
 		(lib_id "NC7WZ07P6X:NC7WZ07P6X_modified")
 		(at 119.38 124.46 0)
@@
 		(fields_autoplaced yes)
 		(property "Reference" "U21"
-			(at 115.57 131.4449 0)
+			(at 116.84 116.84 0)
 			(effects
 				(font
 					(size 1.27 1.27)
 				)
-				(justify left)
 			)
 		)
 		(property "Value" "NC7WZ07P6X"
-			(at 115.57 133.9849 0)
+			(at 116.84 119.38 0)
 			(effects
 				(font
 					(size 1.27 1.27)
 				)
-				(justify left)
 			)
 		)
