File: FPGA-BOARDver3/AUDIO.kicad_sch (KiCad schematic)
At the start: 49 parts, among them J15 5787834-1, J9 SJ1-3525NG, Q10 DMG2305UX-13, U21 NC7WZ07P6X, U24 DSC1033BC1-026.0000, U25 TPS2051BDBVR, U26 TUSB1210BRHBT, U3 AD8592ARM, U35 TPD4E05U06DQAR

Commit message: updated schematic and layout
Parts:
- removed J15: 5787834-1, footprints:CONN4_5787834-1_TEC, symbol 5787834:5787834-1
- removed U24: DSC1033BC1-026.0000, footprints:QFN4_5X3P2_MCH, symbol DSC1033BC1:DSC1033BC1-026.0000
- removed U3: AD8592ARM, footprints:RM_10_ADI, symbol AD8592ARM:AD8592ARM
- added CR5: 7M-26.000MAAJ-T, footprints:CRYSTAL_TXC_7M, symbol 7M_26_000MAAJ_T:7M-26.000MAAJ-T
- added J15: USB-A-S-X-X-SM2, footprints:SAMTEC_USB-A-S-X-X-SM2, symbol USB-A-S-X-X-SM2:USB-A-S-X-X-SM2
- added U10: AD8647ARMZ-REEL, footprints:RM_10_ADI, symbol AD8647ARMZ:AD8647ARMZ-REEL
- C1, C187, C189, C190, C191, C2: LCSC PN (none) -> c1525
- C175, C178: LCSC PN (none) -> c76947
- C177: LCSC PN (none) -> c76951
- C179: footprint footprints:C_0402 -> footprints:C_0805; LCSC PN (none) -> c141660
- C181: LCSC PN (none) -> c14442
- C182: LCSC PN (none) -> c14445
- C183, C186: LCSC PN (none) -> c71687
- C184: LCSC PN (none) -> c15195
- C185: LCSC PN (none) -> c368809
- C188: LCSC PN (none) -> c170151
- C3: LCSC PN (none) -> c307452
- CR3: LCSC PN (none) -> C460860
- F2: LCSC PN (none) -> C133974
- J9: footprint footprints:SJ1-3525NG_CUD -> footprints:CUI_SJ1-3525NG
- Q10: footprint DMG2305UX_13:SOT91P240X110-3N -> footprints:DMG2305UX_13; LCSC PN (none) -> C144153
- R10, R196: LCSC PN (none) -> C60488
- R11, R193: LCSC PN (none) -> C60490
- R12: LCSC PN (none) -> C852482
- R16, R200, R201, R204, R205, R3: LCSC PN (none) -> C106231
- R194, R195: LCSC PN (none) -> C155697
- R197: LCSC PN (none) -> C60491
- R198: LCSC PN (none) -> C138033
- R199: LCSC PN (none) -> c138006
- R202: LCSC PN (none) -> C105871
- R203: LCSC PN (none) -> C106235
- R9: LCSC PN (none) -> C185455
- U21: LCSC PN (none) -> C95342
- U25: LCSC PN (none) -> C24593
- U26: LCSC PN (none) -> C2671015
- U35: LCSC PN (none) -> C138714
Connections:
- net +3V3: now also CR5.1 (VDD), CR5.4
- net AUD_SD: now also U10.5 (*SDA), U10.6 (*SDB)
- net AVCC3V3: now also U10.10 (V+)
- net GNDREF: now also CR5.2 (GND), J15.04 (GND), U10.4 (V-)
- net USBHOST_N: now also U35.2 (D1-), J15.02 (D-); no longer U35.4 (D2+)
- net USBHOST_P: now also U35.1 (D1+), J15.03 (D+); no longer U35.5 (D2-)
- net USBHOST_VBUS: now also U35.4 (D2+), J15.01 (VCC); no longer U35.2 (D1-)
- net USB_SHIELD: now also J15.S1 (SHIELD), J15.S2 (SHIELD__1)
- net at C178.2, C179.1: now also U10.8 (-), U10.9
- net at C3.1, R12.2: now also U10.2 (+)
- net at C177.1, R195.1: now also U10.7 (+)
- net at C175.2, R16.2, R194.2: now also U10.1
- net at R16.1, R193.2: now also U10.3 (-)
- net at R201.1: now also CR5.3 (OUTPUT)
Other:
- moved on the sheet: C184, R201
