File: FPGA-BOARDver3/FPGA_POWER.kicad_sch (KiCad schematic)
At the start: 56 parts, among them U21 XC7Z020-1CLG400I_

Commit message: assigned footprints for power section and ddr3
Parts:
- C100, C101, C102, C103, C104, C105, C106, C107, C108, C109, C110, C111, C112, C113, C114, C115, C116, C117, C118, C119, C120, C121, C122, C123, C124, C125, C126, C127, C128, C129, C130, C131, C132, C133, C134, C135, C136, C137, C138, C85, C86, C87, C88, C89, C90, C91, C92, C93, C94, C95, C96, C97, C98, C99: footprint (none) -> JLCPCB:C_0402
- U21: footprint CLG400_ZYNQ-7000_AMD -> XC7Z020-1CLG400I:CLG400_ZYNQ-7000_AMD

Commit message: footprints added to project specific library
Parts:
- C100, C101, C102, C103, C104, C105, C106, C107, C108, C109, C110, C111, C112, C113, C114, C115, C116, C117, C118, C119, C120, C121, C122, C123, C124, C125, C126, C127, C128, C129, C130, C131, C132, C133, C134, C135, C136, C137, C138, C85, C86, C87, C88, C89, C90, C91, C92, C93, C94, C95, C96, C97, C98, C99: footprint JLCPCB:C_0402 -> footprints:C_0402
- FL1: footprint BLM18AG601SZ1D:BEADC1608X95N -> footprints:BEADC1608X95N
- U21: footprint XC7Z020-1CLG400I:CLG400_ZYNQ-7000_AMD -> footprints:CLG400_ZYNQ-7000_AMD
Changed lines of the file:
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@@
 			)
 		)
-		(property "Footprint" "JLCPCB:C_0402"
+		(property "Footprint" "footprints:C_0402"
 			(at 103.8352 92.71 0)
 			(effects
@@
 			)
 		)
-		(property "Footprint" "JLCPCB:C_0402"
+		(property "Footprint" "footprints:C_0402"
 			(at 227.0252 57.15 0)
 			(effects
@@
 			)
 		)
-		(property "Footprint" "JLCPCB:C_0402"
+		(property "Footprint" "footprints:C_0402"
 			(at 103.8352 62.23 0)
 			(effects
@@
 			)
 		)
-		(property "Footprint" "JLCPCB:C_0402"
+		(property "Footprint" "footprints:C_0402"
 			(at 207.9752 57.15 0)
 			(effects
@@
 			)
 		)
-		(property "Footprint" "JLCPCB:C_0402"
+		(property "Footprint" "footprints:C_0402"
 			(at 199.0852 114.3 0)
 			(effects
@@
 			)
 		)
-		(property "Footprint" "JLCPCB:C_0402"
+		(property "Footprint" "footprints:C_0402"
 			(at 86.0552 77.47 0)
 			(effects
@@
 			)
 		)
-		(property "Footprint" "JLCPCB:C_0402"
+		(property "Footprint" "footprints:C_0402"
 			(at 94.9452 77.47 0)
 			(effects
@@
 			)
 		)
-		(property "Footprint" "JLCPCB:C_0402"
+		(property "Footprint" "footprints:C_0402"
 			(at 218.1352 57.15 0)
 			(effects
@@
 			)
 		)
-		(property "Footprint" "JLCPCB:C_0402"
+		(property "Footprint" "footprints:C_0402"
 			(at 188.9252 114.3 0)
 			(effects
@@
 			)
 		)
-		(property "Footprint" "XC7Z020-1CLG400I:CLG400_ZYNQ-7000_AMD"
+		(property "Footprint" "footprints:CLG400_ZYNQ-7000_AMD"
 			(at 40.132 166.878 0)
 			(effects
@@
 			)
 		)
-		(property "Footprint" "JLCPCB:C_0402"
+		(property "Footprint" "footprints:C_0402"
 			(at 190.1952 41.91 0)
 			(effects
@@
 			)
 		)
-		(property "Footprint" "JLCPCB:C_0402"
+		(property "Footprint" "footprints:C_0402"
 			(at 86.0552 62.23 0)
 			(effects
@@
 			)
 		)
-		(property "Footprint" "JLCPCB:C_0402"
+		(property "Footprint" "footprints:C_0402"
 			(at 94.9452 92.71 0)
 			(effects
@@
 			)
 		)
-		(property "Footprint" "JLCPCB:C_0402"
+		(property "Footprint" "footprints:C_0402"
 			(at 190.1952 57.15 0)
 			(effects
@@
 			)
 		)
-		(property "Footprint" "JLCPCB:C_0402"
+		(property "Footprint" "footprints:C_0402"
 			(at 237.1852 74.93 0)
 			(effects
@@
 			)
 		)
-		(property "Footprint" "JLCPCB:C_0402"
+		(property "Footprint" "footprints:C_0402"
 			(at 94.9452 36.83 0)
 			(effects
@@
 			)
 		)
-		(property "Footprint" "JLCPCB:C_0402"
+		(property "Footprint" "footprints:C_0402"
 			(at 227.0252 114.3 0)
 			(effects
@@
 			)
 		)
-		(property "Footprint" "BLM18AG601SZ1D:BEADC1608X95N"
+		(property "Footprint" "footprints:BEADC1608X95N"
 			(at 241.3 138.43 0)
 			(effects
@@
 			)
 		)
-		(property "Footprint" "JLCPCB:C_0402"
+		(property "Footprint" "footprints:C_0402"
 			(at 188.9252 97.79 0)
 			(effects
@@
 			)
 		)
-		(property "Footprint" "JLCPCB:C_0402"
+		(property "Footprint" "footprints:C_0402"
 			(at 237.1852 57.15 0)
 			(effects
@@
 			)
 		)
-		(property "Footprint" "JLCPCB:C_0402"
+		(property "Footprint" "footprints:C_0402"
 			(at 216.8652 114.3 0)
 			(effects
@@
 			)
 		)
-		(property "Footprint" "XC7Z020-1CLG400I:CLG400_ZYNQ-7000_AMD"
+		(property "Footprint" "footprints:CLG400_ZYNQ-7000_AMD"
 			(at 135.382 41.402 0)
 			(effects
@@
 			)
 		)
-		(property "Footprint" "JLCPCB:C_0402"
+		(property "Footprint" "footprints:C_0402"
 			(at 67.0052 109.22 0)
 			(effects
@@
 			)
 		)
-		(property "Footprint" "JLCPCB:C_0402"
+		(property "Footprint" "footprints:C_0402"
 			(at 86.0552 124.46 0)
 			(effects
@@
 			)
 		)
-		(property "Footprint" "JLCPCB:C_0402"
+		(property "Footprint" "footprints:C_0402"
 			(at 237.1852 114.3 0)
 			(effects
@@
 			)
 		)
-		(property "Footprint" "JLCPCB:C_0402"
+		(property "Footprint" "footprints:C_0402"
 			(at 199.0852 74.93 0)
 			(effects
@@
 			)
 		)
-		(property "Footprint" "JLCPCB:C_0402"
+		(property "Footprint" "footprints:C_0402"
 			(at 180.0352 114.3 0)
 			(effects
@@
 			)
 		)
-		(property "Footprint" "JLCPCB:C_0402"
+		(property "Footprint" "footprints:C_0402"
 			(at 207.9752 114.3 0)
 			(effects
@@
 			)
 		)
-		(property "Footprint" "JLCPCB:C_0402"
+		(property "Footprint" "footprints:C_0402"
 			(at 180.0352 41.91 0)
 			(effects
@@
 			)
 		)
-		(property "Footprint" "JLCPCB:C_0402"
+		(property "Footprint" "footprints:C_0402"
 			(at 94.9452 124.46 0)
 			(effects
@@
 			)
 		)
-		(property "Footprint" "JLCPCB:C_0402"
+		(property "Footprint" "footprints:C_0402"
 			(at 180.0352 74.93 0)
 			(effects
@@
 			)
 		)
-		(property "Footprint" "JLCPCB:C_0402"
+		(property "Footprint" "footprints:C_0402"
 			(at 75.8952 36.83 0)
 			(effects
@@
 			)
 		)
-		(property "Footprint" "JLCPCB:C_0402"
+		(property "Footprint" "footprints:C_0402"
 			(at 103.8352 36.83 0)
 			(effects
@@
 			)
 		)
-		(property "Footprint" "JLCPCB:C_0402"
+		(property "Footprint" "footprints:C_0402"
 			(at 190.1952 74.93 0)
 			(effects
@@
 			)
 		)
-		(property "Footprint" "JLCPCB:C_0402"
+		(property "Footprint" "footprints:C_0402"
 			(at 199.0852 97.79 0)
 			(effects
@@
 			)
 		)
-		(property "Footprint" "JLCPCB:C_0402"
+		(property "Footprint" "footprints:C_0402"
 			(at 199.0852 57.15 0)
 			(effects
@@
 			)
 		)
-		(property "Footprint" "JLCPCB:C_0402"
+		(property "Footprint" "footprints:C_0402"
 			(at 254.9652 38.1 0)
 			(effects
@@
 			)
 		)
-		(property "Footprint" "JLCPCB:C_0402"
+		(property "Footprint" "footprints:C_0402"
 			(at 86.0552 36.83 0)
 			(effects
@@
 			)
 		)
-		(property "Footprint" "JLCPCB:C_0402"
+		(property "Footprint" "footprints:C_0402"
 			(at 199.0852 41.91 0)
 			(effects
@@
 			)
 		)
-		(property "Footprint" "JLCPCB:C_0402"
+		(property "Footprint" "footprints:C_0402"
 			(at 87.3252 109.22 0)
 			(effects
@@
 			)
 		)
-		(property "Footprint" "JLCPCB:C_0402"
+		(property "Footprint" "footprints:C_0402"
 			(at 207.9752 41.91 0)
 			(effects
@@
 			)
 		)
-		(property "Footprint" "JLCPCB:C_0402"
+		(property "Footprint" "footprints:C_0402"
 			(at 180.0352 97.79 0)
 			(effects
@@
 			)
 		)
-		(property "Footprint" "JLCPCB:C_0402"
+		(property "Footprint" "footprints:C_0402"
 			(at 94.9452 62.23 0)
 			(effects
@@
 			)
 		)
-		(property "Footprint" "JLCPCB:C_0402"
+		(property "Footprint" "footprints:C_0402"
 			(at 56.8452 36.83 0)
 			(effects
@@
 			)
 		)
-		(property "Footprint" "JLCPCB:C_0402"
+		(property "Footprint" "footprints:C_0402"
 			(at 94.9452 109.22 0)
 			(effects
@@
 			)
 		)
-		(property "Footprint" "JLCPCB:C_0402"
+		(property "Footprint" "footprints:C_0402"
 			(at 220.6752 147.32 0)
 			(effects
@@
 			)
 		)
-		(property "Footprint" "JLCPCB:C_0402"
+		(property "Footprint" "footprints:C_0402"
 			(at 180.0352 57.15 0)
 			(effects
@@
 			)
 		)
-		(property "Footprint" "JLCPCB:C_0402"
+		(property "Footprint" "footprints:C_0402"
 			(at 103.8352 109.22 0)
 			(effects
@@
 			)
 		)
-		(property "Footprint" "JLCPCB:C_0402"
+		(property "Footprint" "footprints:C_0402"
 			(at 67.0052 36.83 0)
 			(effects
@@
 			)
 		)
-		(property "Footprint" "JLCPCB:C_0402"
+		(property "Footprint" "footprints:C_0402"
 			(at 86.0552 92.71 0)
 			(effects
@@
 			)
 		)
-		(property "Footprint" "JLCPCB:C_0402"
+		(property "Footprint" "footprints:C_0402"
 			(at 103.8352 77.47 0)
 			(effects
@@
 			)
 		)
-		(property "Footprint" "JLCPCB:C_0402"
+		(property "Footprint" "footprints:C_0402"
 			(at 103.8352 124.46 0)
 			(effects
@@
 			)
 		)
-		(property "Footprint" "JLCPCB:C_0402"
+		(property "Footprint" "footprints:C_0402"
 			(at 77.1652 109.22 0)
 			(effects
@@
 			)
 		)
-		(property "Footprint" "JLCPCB:C_0402"
+		(property "Footprint" "footprints:C_0402"
 			(at 227.0252 74.93 0)
 			(effects
@@
 			)
 		)
-		(property "Footprint" "JLCPCB:C_0402"
+		(property "Footprint" "footprints:C_0402"
 			(at 207.9752 74.93 0)
 			(effects
@@
 			)
 		)
-		(property "Footprint" "JLCPCB:C_0402"
+		(property "Footprint" "footprints:C_0402"
 			(at 207.9752 147.32 0)
 			(effects
@@
 			)
 		)
-		(property "Footprint" "JLCPCB:C_0402"
+		(property "Footprint" "footprints:C_0402"
 			(at 216.8652 74.93 0)
 			(effects

Commit message: added fpga banks and final fpga symbol
Parts:
- removed U21: XC7Z020-1CLG400I_, footprints:CLG400_ZYNQ-7000_AMD, symbol 2025-03-16_22-31-30:XC7Z020-1CLG400I_
- added U1: XC7Z020-1CLG400I__, footprints:CLG400_ZYNQ-7000_AMD, symbol xc7z020-1clg400i_complete:XC7Z020-1CLG400I__
Connections:
- net +1V0: now also U1.G11 (VCCBRAM), U1.G7 (VCCPINT), U1.H10 (VCCBRAM), U1.J7 (VCCPINT), U1.L7 (VCCPINT), U1.N7 (VCCPINT), U1.P8 (VCCPINT), U1.R13 (VCCINT), U1.R7 (VCCPINT)
- net +1V5: now also U1.A3 (VCCO_DDR_502), U1.D2 (VCCO_DDR_502), U1.E5 (VCCO_DDR_502), U1.G1 (VCCO_DDR_502), U1.H4 (VCCO_DDR_502), U1.L3 (VCCO_DDR_502), U1.P2 (VCCO_DDR_502), U1.R5 (VCCO_DDR_502), U1.U1 (VCCO_DDR_502), U1.V4 (VCCO_DDR_502)
- net +1V8: now also U1.A13 (VCCO_MIO1_501), U1.B16 (VCCO_MIO1_501), U1.D12 (VCCO_MIO1_501), U1.E15 (VCCO_MIO1_501), U1.F11 (VCCBATT_0), U1.F8 (VCCPAUX), U1.G9 (VCCPAUX), U1.H8 (VCCPAUX), U1.J11 (VCCAUX), U1.K8 (VCCPAUX), U1.L11 (VCCAUX), U1.M8 (VCCPAUX), U1.N11 (VCCAUX), U1.N9 (VCCAUX), U1.P10 (VCCAUX), U1.R9 (VCCAUX)
- net +3V3: now also U1.B6 (VCCO_MIO0_500), U1.C19 (VCCO_35), U1.D7 (VCCO_MIO0_500), U1.F18 (VCCO_35), U1.H14 (VCCO_35), U1.J17 (VCCO_35), U1.K20 (VCCO_35), U1.K6 (VCCO_0), U1.M16 (VCCO_35), U1.N19 (VCCO_34), U1.R15 (VCCO_34), U1.T18 (VCCO_34), U1.T8 (VCCO_13), U1.U11 (VCCO_13), U1.V14 (VCCO_34), U1.W17 (VCCO_34), U1.W7 (VCCO_13), U1.Y10 (VCCO_13), U1.Y20 (VCCO_34)
- net GNDREF: now also U1.A18 (GND), U1.A8 (GND), U1.B1 (GND), U1.B11 (GND), U1.C14 (GND), U1.C4 (GND), U1.C9 (GND), U1.D17 (GND), U1.E10 (GND), U1.E20 (GND), U1.F3 (GND), U1.F7 (GND), U1.G10 (GND), U1.G12 (GND), U1.G16 (GND), U1.H11 (GND), U1.H13 (GND), U1.H19 (GND), U1.H7 (GND), U1.H9 (GND), U1.J12 (GND), U1.J2 (GND), U1.J8 (GND), U1.K11 (GND), U1.K13 (GND), U1.K15 (GND), U1.K5 (GND), U1.K7 (GND), U1.L12 (GND), U1.L18 (GND), U1.L8 (GND), U1.M1 (GND), U1.M11 (GND), U1.M13 (GND), U1.M7 (GND), U1.N10 (GND), U1.N12 (GND), U1.N14 (GND), U1.N4 (GND), U1.N8 (GND), U1.P11 (GND), U1.P13 (GND), U1.P17 (GND), U1.P7 (GND), U1.P9 (GND), U1.R12 (GND), U1.R20 (GND), U1.R8 (GND), U1.T13 (GND), U1.T3 (GND), U1.T7 (GND), U1.U16 (GND), U1.U6 (GND), U1.V19 (GND), U1.V9 (GND), U1.W12 (GND), U1.W2 (GND), U1.Y15 (GND), U1.Y5 (GND)
- net VCCPLL: now also U1.G8 (VCCPLL)

Commit message: spdif fpga bansks
Parts:
- U1: footprint footprints:CLG400_ZYNQ-7000_AMD -> XC7Z020-1CLG400I:CLG400_ZYNQ-7000_AMD

Commit message: All pages complete , pi header left
Parts:
- U1: footprint XC7Z020-1CLG400I:CLG400_ZYNQ-7000_AMD -> footprints:CLG400_ZYNQ-7000_AMD
Changed lines of the file:
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@@
 	)
 	(symbol
+		(lib_name "XC7Z020-1CLG400I___1")
 		(lib_id "xc7z020-1clg400i_complete:XC7Z020-1CLG400I__")
 		(at 115.57 29.21 0)
@@
 		(fields_autoplaced yes)
 		(property "Reference" "U1"
-			(at 140.97 19.05 0)
+			(at 163.195 12.7 0)
 			(effects
 				(font
@@
 		)
 		(property "Value" "XC7Z020-1CLG400I__"
-			(at 140.97 21.59 0)
+			(at 163.195 15.24 0)
 			(effects
 				(font
@@
 			)
 		)
-		(property "Footprint" "XC7Z020-1CLG400I:CLG400_ZYNQ-7000_AMD"
+		(property "Footprint" "footprints:CLG400_ZYNQ-7000_AMD"
 			(at 149.098 -48.26 0)
 			(effects
@@
 					(unit 6)
 				)
+				(path "/4a327bdf-04e5-4836-9c0a-5fb801c23f64/41e60eaf-6223-4c1c-9aff-98af239c75fe"
+					(reference "U1")
+					(unit 6)
+				)
 			)
 		)
@@
 		(fields_autoplaced yes)
 		(property "Reference" "U1"
-			(at 21.59 165.0999 90)
+			(at 11.43 139.065 0)
 			(effects
 				(font
 					(size 1.524 1.524)
 				)
-				(justify left)
 			)
 		)
 		(property "Value" "XC7Z020-1CLG400I__"
-			(at 21.59 167.6399 90)
+			(at 13.97 139.065 0)
 			(effects
 				(font
 					(size 1.524 1.524)
 				)
-				(justify left)
 			)
 		)
-		(property "Footprint" "XC7Z020-1CLG400I:CLG400_ZYNQ-7000_AMD"
+		(property "Footprint" "footprints:CLG400_ZYNQ-7000_AMD"
 			(at -49.53 153.162 0)
 			(effects
@@
 					(reference "U1")
 					(unit 7)
+				)
+				(path "/4a327bdf-04e5-4836-9c0a-5fb801c23f64/41e60eaf-6223-4c1c-9aff-98af239c75fe"
+					(reference "U1")
+					(unit 7)

Commit message: added audio out and usb
Parts:
- C138: value 100uF -> 47uF
Connections:
- net +1V8: no longer C116.1, C130.1, C93.1, U1.A13 (VCCO_MIO1_501), U1.B16 (VCCO_MIO1_501), U1.D12 (VCCO_MIO1_501), U1.E15 (VCCO_MIO1_501)
- new net VCC1V8_IO: C116.1, C130.1, C93.1, U1.A13 (VCCO_MIO1_501), U1.B16 (VCCO_MIO1_501), U1.D12 (VCCO_MIO1_501), U1.E15 (VCCO_MIO1_501)

Commit message: updated schematic and layout
Parts:
- C100, C101, C102, C103, C104, C105, C106, C107, C108, C109, C110, C111, C112, C113, C87, C88, C89, C90, C91, C92, C93, C94, C95, C96, C97, C98, C99: LCSC PN (none) -> c92361
- C114, C115, C117, C118, C119, C120, C121, C122, C123, C124, C126, C127, C86: LCSC PN (none) -> c23733
- C116: LCSC PN (none) -> c84705
- C125, C138: footprint footprints:C_0402 -> footprints:C_0805; LCSC PN (none) -> c16790
- C128, C129, C130, C131, C132, C133, C134, C135, C136, C85: footprint footprints:C_0402 -> footprints:C_0805; LCSC PN (none) -> c141660
- C137: LCSC PN (none) -> c315248
- FL1: LCSC PN (none) -> digi/mouser
- U1: LCSC PN (none) -> C1519081
Connections:
- net +1V0: now also U1.G13 (VCCINT), U1.H12 (VCCINT), U1.J13 (VCCINT), U1.K12 (VCCINT), U1.L13 (VCCINT), U1.M12 (VCCINT), U1.N13 (VCCINT), U1.P12 (VCCINT)
