File: FPGA-BOARDver3/HDMI.kicad_sch (KiCad schematic)
At the start: 47 parts, among them J10 10029449-001RLF, J11 10029449-001RLF, Q9 FDV301N, U10 GTL2002GM, U11 NC7SZ125M5X, U8 GTL2002GM

Commit message: added audio out and usb
Parts:
- added R207: 10K, footprints:R_0402, symbol Device:R_US
- R127, R128, R129, R130: value 1.5K -> 1K
- R152: value 49.9 -> 1K
Connections:
- net HDMI_RX_5V0: now also R131.2, R132.2, R133.2
- net HDMI_RX_SCL: now also U8.3 (S1); no longer U8.5 (D2)
- net HDMI_RX_SCL_LS: now also U8.5 (D2); no longer U8.3 (S1)
- net HDMI_RX_SDA: now also U8.4 (S2); no longer U8.6 (D1)
- net HDMI_RX_SDA_LS: now also U8.6 (D1); no longer U8.4 (S2)
- net HDMI_TX_5V0: no longer R131.2, R132.2, R133.2
- net HDMI_TX_SCL: now also U10.3 (S1); no longer U10.5 (D2)
- net HDMI_TX_SCL_LS: now also U10.5 (D2); no longer U10.3 (S1)
- net HDMI_TX_SDA: now also U10.4 (S2); no longer U10.6 (D1)
- net HDMI_TX_SDA_LS: now also U10.6 (D1); no longer U10.4 (S2)
- net at J10.19, R154.2: now also R207.2; no longer Q9.1
- new net: Q9.1, R207.1

Commit message: updated schematic and layout
Parts:
- removed U10, U8: GTL2002GM, footprints:SOT902-1_NXP, symbol GTL2002GM:GTL2002GM
- added R240, R241: 200k, footprints:R_0402, symbol Device:R_US
- added U24, U8: TXS0102DCUR, footprints:SOP50P310X90-8N, symbol TXS0102DCUR:TXS0102DCUR
- C17, C22, C23, C24, C25: LCSC PN (none) -> c1525
- C52: footprint footprints:C_0402 -> footprints:C_1808_4520Metric; LCSC PN (none) -> c237595
- D26, D27: LCSC PN (none) -> C152479
- F1: footprint footprints:FUSE_PTS1206_EAT -> footprints:PTS120630V012; LCSC PN (none) -> C2442491
- J10, J11: LCSC PN (none) -> C428493
- Q9: LCSC PN (none) -> C15310
- R124, R131: value 200K -> 10K; LCSC PN (none) -> C60490
- R125, R126, R132, R133: LCSC PN (none) -> C114759
- R127, R128, R129, R130, R152: LCSC PN (none) -> C106235
- R134, R135, R136, R137, R138, R139, R140, R141, R144, R145, R146, R147, R148, R149, R150, R151: LCSC PN (none) -> C87044
- R142, R143: LCSC PN (none) -> C138022
- R153: LCSC PN (none) -> C138033
- R154, R207: LCSC PN (none) -> C60490
- R155: LCSC PN (none) -> C105871
- U11: LCSC PN (none) -> C7420
Connections:
- net +3V3: now also R124.1, R131.1, U24.3 (VCCA), U8.3 (VCCA)
- net GNDREF: now also U24.2 (GND), U8.2 (GND)
- net HDMI_RX_5V0: now also R241.1; no longer R131.2
- net HDMI_RX_SCL: now also U24.5 (A1)
- net HDMI_RX_SCL_LS: now also R132.1, U24.8 (B1); no longer R133.1
- net HDMI_RX_SDA: now also U24.4 (A2)
- net HDMI_RX_SDA_LS: now also R133.1, U24.1 (B2); no longer R132.1
- net HDMI_TX_5V0: now also R240.1; no longer R124.2
- net HDMI_TX_SCL: now also U8.5 (A1)
- net HDMI_TX_SCL_LS: now also R125.1, U8.8 (B1); no longer R126.1
- net HDMI_TX_SDA: now also U8.4 (A2)
- net HDMI_TX_SDA_LS: now also R126.1, U8.1 (B2); no longer R125.1
- net at C17.1: now also R240.2, U8.7 (VCCB); no longer R124.1
- net at C24.1: now also R241.2, U24.7 (VCCB); no longer R131.1
- new net: R131.2, U8.6 (OE)
- new net: R124.2, U24.6 (OE)
Other:
- moved on the sheet: F1
