File: FPGA-BOARDver3/PMOD,LED,SWITCHES.kicad_sch (KiCad schematic)
At the start: 86 parts, among them P1 PMOD-Device-x2-Type-Generic-A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, P2 PMOD-Device-x2-Type-Generic-A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, Q1 BC107, Q2 BC107, Q3 BC107, Q4 BC107, Q5 BC107, Q6 BC107, SW2 SW_Push, SW3 SW_Push, SW4 SW_Push, SW5 SW_Push, SW6 SW_SP3T, SW7 SW_SP3T

Commit message: footprints added to project specific library
Parts:
- C6, C7: footprint JLCPCB:C_0402 -> footprints:C_0402
- D10, D11, D12, D13, D14, D15, D16, D17, D18, D19, D20, D21, D22, D23, D24, D9: footprint BZT52C5V1_7_F:SOD123_DIO -> footprints:SOD123_DIO
- D7, D8: footprint SMLVN6RBG1U1:LED_SMLV56_ROM -> footprints:LED_SMLV56_ROM
- R1, R13, R14, R15, R2, R21, R22, R23, R24, R25, R26, R27, R28, R29, R30, R31, R32, R33, R34, R35, R55, R56, R57, R58, R59, R60, R61, R62, R63, R64, R65, R66, R67, R68, R69, R70, R71, R72, R73, R74, R75, R76, R77, R78, R79, R80, R81, R82: footprint JLCPCB:R_0402 -> footprints:R_0402
Changed lines of the file:
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@@
 			)
 		)
-		(property "Footprint" "JLCPCB:R_0402"
+		(property "Footprint" "footprints:R_0402"
 			(at 139.954 162.814 90)
 			(effects
@@
 			)
 		)
-		(property "Footprint" "JLCPCB:R_0402"
+		(property "Footprint" "footprints:R_0402"
 			(at 105.156 32.004 90)
 			(effects
@@
 			)
 		)
-		(property "Footprint" "JLCPCB:R_0402"
+		(property "Footprint" "footprints:R_0402"
 			(at 214.884 58.166 90)
 			(effects
@@
 			)
 		)
-		(property "Footprint" "JLCPCB:R_0402"
+		(property "Footprint" "footprints:R_0402"
 			(at 156.464 24.384 90)
 			(effects
@@
 			)
 		)
-		(property "Footprint" "JLCPCB:R_0402"
+		(property "Footprint" "footprints:R_0402"
 			(at 214.884 108.966 90)
 			(effects
@@
 			)
 		)
-		(property "Footprint" "BZT52C5V1_7_F:SOD123_DIO"
+		(property "Footprint" "footprints:SOD123_DIO"
 			(at 93.98 92.71 0)
 			(effects
@@
 			)
 		)
-		(property "Footprint" "BZT52C5V1_7_F:SOD123_DIO"
+		(property "Footprint" "footprints:SOD123_DIO"
 			(at 90.17 44.45 0)
 			(effects
@@
 			)
 		)
-		(property "Footprint" "JLCPCB:R_0402"
+		(property "Footprint" "footprints:R_0402"
 			(at 38.354 157.734 90)
 			(effects
@@
 			)
 		)
-		(property "Footprint" "JLCPCB:R_0402"
+		(property "Footprint" "footprints:R_0402"
 			(at 105.156 35.814 90)
 			(effects
@@
 			)
 		)
-		(property "Footprint" "JLCPCB:C_0402"
+		(property "Footprint" "footprints:C_0402"
 			(at 152.0952 44.45 0)
 			(effects
@@
 			)
 		)
-		(property "Footprint" "BZT52C5V1_7_F:SOD123_DIO"
+		(property "Footprint" "footprints:SOD123_DIO"
 			(at 41.91 92.71 0)
 			(effects
@@
 			)
 		)
-		(property "Footprint" "SMLVN6RBG1U1:LED_SMLV56_ROM"
+		(property "Footprint" "footprints:LED_SMLV56_ROM"
 			(at 171.45 90.17 0)
 			(effects
@@
 			)
 		)
-		(property "Footprint" "JLCPCB:R_0402"
+		(property "Footprint" "footprints:R_0402"
 			(at 105.156 28.194 90)
 			(effects
@@
 			)
 		)
-		(property "Footprint" "JLCPCB:R_0402"
+		(property "Footprint" "footprints:R_0402"
 			(at 29.464 24.384 90)
 			(effects
@@
 			)
 		)
-		(property "Footprint" "JLCPCB:R_0402"
+		(property "Footprint" "footprints:R_0402"
 			(at 236.474 58.166 90)
 			(effects
@@
 			)
 		)
-		(property "Footprint" "JLCPCB:R_0402"
+		(property "Footprint" "footprints:R_0402"
 			(at 156.464 80.264 90)
 			(effects
@@
 			)
 		)
-		(property "Footprint" "JLCPCB:R_0402"
+		(property "Footprint" "footprints:R_0402"
 			(at 200.914 85.344 90)
 			(effects
@@
 			)
 		)
-		(property "Footprint" "JLCPCB:R_0402"
+		(property "Footprint" "footprints:R_0402"
 			(at 200.914 19.304 90)
 			(effects
@@
 			)
 		)
-		(property "Footprint" "JLCPCB:R_0402"
+		(property "Footprint" "footprints:R_0402"
 			(at 33.274 72.644 90)
 			(effects
@@
 			)
 		)
-		(property "Footprint" "JLCPCB:R_0402"
+		(property "Footprint" "footprints:R_0402"
 			(at 121.666 170.434 90)
 			(effects
@@
 			)
 		)
-		(property "Footprint" "JLCPCB:R_0402"
+		(property "Footprint" "footprints:R_0402"
 			(at 157.734 34.544 90)
 			(effects
@@
 			)
 		)
-		(property "Footprint" "JLCPCB:R_0402"
+		(property "Footprint" "footprints:R_0402"
 			(at 139.954 142.494 90)
 			(effects
@@
 			)
 		)
-		(property "Footprint" "JLCPCB:R_0402"
+		(property "Footprint" "footprints:R_0402"
 			(at 200.914 70.104 90)
 			(effects
@@
 			)
 		)
-		(property "Footprint" "JLCPCB:R_0402"
+		(property "Footprint" "footprints:R_0402"
 			(at 29.464 32.004 90)
 			(effects
@@
 			)
 		)
-		(property "Footprint" "JLCPCB:R_0402"
+		(property "Footprint" "footprints:R_0402"
 			(at 139.954 152.654 90)
 			(effects
@@
 			)
 		)
-		(property "Footprint" "BZT52C5V1_7_F:SOD123_DIO"
+		(property "Footprint" "footprints:SOD123_DIO"
 			(at 38.1 44.45 0)
 			(effects
@@
 			)
 		)
-		(property "Footprint" "JLCPCB:R_0402"
+		(property "Footprint" "footprints:R_0402"
 			(at 38.354 146.304 90)
 			(effects
@@
 			)
 		)
-		(property "Footprint" "JLCPCB:R_0402"
+		(property "Footprint" "footprints:R_0402"
 			(at 221.234 145.034 90)
 			(effects
@@
 			)
 		)
-		(property "Footprint" "JLCPCB:R_0402"
+		(property "Footprint" "footprints:R_0402"
 			(at 37.084 169.164 90)
 			(effects
@@
 			)
 		)
-		(property "Footprint" "JLCPCB:R_0402"
+		(property "Footprint" "footprints:R_0402"
 			(at 29.464 35.814 90)
 			(effects
@@
 			)
 		)
-		(property "Footprint" "JLCPCB:R_0402"
+		(property "Footprint" "footprints:R_0402"
 			(at 33.274 80.264 90)
 			(effects
@@
 			)
 		)
-		(property "Footprint" "JLCPCB:R_0402"
+		(property "Footprint" "footprints:R_0402"
 			(at 108.966 84.074 90)
 			(effects
@@
 			)
 		)
-		(property "Footprint" "BZT52C5V1_7_F:SOD123_DIO"
+		(property "Footprint" "footprints:SOD123_DIO"
 			(at 82.55 44.45 0)
 			(effects
@@
 			)
 		)
-		(property "Footprint" "JLCPCB:R_0402"
+		(property "Footprint" "footprints:R_0402"
 			(at 200.914 49.784 90)
 			(effects
@@
 			)
 		)
-		(property "Footprint" "JLCPCB:R_0402"
+		(property "Footprint" "footprints:R_0402"
 			(at 103.886 170.434 90)
 			(effects
@@
 			)
 		)
-		(property "Footprint" "BZT52C5V1_7_F:SOD123_DIO"
+		(property "Footprint" "footprints:SOD123_DIO"
 			(at 86.36 44.45 0)
 			(effects
@@
 			)
 		)
-		(property "Footprint" "BZT52C5V1_7_F:SOD123_DIO"
+		(property "Footprint" "footprints:SOD123_DIO"
 			(at 86.36 92.71 0)
 			(effects
@@
 			)
 		)
-		(property "Footprint" "JLCPCB:R_0402"
+		(property "Footprint" "footprints:R_0402"
 			(at 156.464 75.184 90)
 			(effects
@@
 			)
 		)
-		(property "Footprint" "BZT52C5V1_7_F:SOD123_DIO"
+		(property "Footprint" "footprints:SOD123_DIO"
 			(at 97.79 92.71 0)
 			(effects
@@
 			)
 		)
-		(property "Footprint" "BZT52C5V1_7_F:SOD123_DIO"
+		(property "Footprint" "footprints:SOD123_DIO"
 			(at 93.98 44.45 0)
 			(effects
@@
 			)
 		)
-		(property "Footprint" "JLCPCB:R_0402"
+		(property "Footprint" "footprints:R_0402"
 			(at 200.914 34.544 90)
 			(effects
@@
 			)
 		)
-		(property "Footprint" "JLCPCB:C_0402"
+		(property "Footprint" "footprints:C_0402"
 			(at 152.0952 95.25 0)
 			(effects
@@
 			)
 		)
-		(property "Footprint" "JLCPCB:R_0402"
+		(property "Footprint" "footprints:R_0402"
 			(at 108.966 72.644 90)
 			(effects
@@
 			)
 		)
-		(property "Footprint" "BZT52C5V1_7_F:SOD123_DIO"
+		(property "Footprint" "footprints:SOD123_DIO"
 			(at 41.91 44.45 0)
 			(effects
@@
 			)
 		)
-		(property "Footprint" "JLCPCB:R_0402"
+		(property "Footprint" "footprints:R_0402"
 			(at 108.966 80.264 90)
 			(effects
@@
 			)
 		)
-		(property "Footprint" "JLCPCB:R_0402"
+		(property "Footprint" "footprints:R_0402"
 			(at 33.274 76.454 90)
 			(effects
@@
 			)
 		)
-		(property "Footprint" "JLCPCB:R_0402"
+		(property "Footprint" "footprints:R_0402"
 			(at 216.154 136.144 90)
 			(effects
@@
 			)
 		)
-		(property "Footprint" "JLCPCB:R_0402"
+		(property "Footprint" "footprints:R_0402"
 			(at 236.474 108.966 90)
 			(effects
@@
 			)
 		)
-		(property "Footprint" "BZT52C5V1_7_F:SOD123_DIO"
+		(property "Footprint" "footprints:SOD123_DIO"
 			(at 49.53 44.45 0)
 			(effects
@@
 			)
 		)
-		(property "Footprint" "JLCPCB:R_0402"
+		(property "Footprint" "footprints:R_0402"
 			(at 33.274 84.074 90)
 			(effects
@@
 			)
 		)
-		(property "Footprint" "BZT52C5V1_7_F:SOD123_DIO"
+		(property "Footprint" "footprints:SOD123_DIO"
 			(at 49.53 92.71 0)
 			(effects
@@
 			)
 		)
-		(property "Footprint" "JLCPCB:R_0402"
+		(property "Footprint" "footprints:R_0402"
 			(at 156.464 29.464 90)
 			(effects
@@
 			)
 		)
-		(property "Footprint" "BZT52C5V1_7_F:SOD123_DIO"
+		(property "Footprint" "footprints:SOD123_DIO"
 			(at 45.72 92.71 0)
 			(effects
@@
 			)
 		)
-		(property "Footprint" "JLCPCB:R_0402"
+		(property "Footprint" "footprints:R_0402"
 			(at 38.354 134.874 90)
 			(effects
@@
 			)
 		)
-		(property "Footprint" "JLCPCB:R_0402"
+		(property "Footprint" "footprints:R_0402"
 			(at 112.776 170.434 90)
 			(effects
@@
 			)
 		)
-		(property "Footprint" "JLCPCB:R_0402"
+		(property "Footprint" "footprints:R_0402"
 			(at 129.286 170.434 90)
 			(effects
@@
 			)
 		)
-		(property "Footprint" "JLCPCB:R_0402"
+		(property "Footprint" "footprints:R_0402"
 			(at 105.156 24.384 90)
 			(effects
@@
 			)
 		)
-		(property "Footprint" "JLCPCB:R_0402"
+		(property "Footprint" "footprints:R_0402"
 			(at 200.914 100.584 90)
 			(effects
@@
 			)
 		)
-		(property "Footprint" "JLCPCB:R_0402"
+		(property "Footprint" "footprints:R_0402"
 			(at 108.966 76.454 90)
 			(effects
@@
 			)
 		)
-		(property "Footprint" "JLCPCB:R_0402"
+		(property "Footprint" "footprints:R_0402"
 			(at 226.314 108.966 90)
 			(effects
@@
 			)
 		)
-		(property "Footprint" "BZT52C5V1_7_F:SOD123_DIO"
+		(property "Footprint" "footprints:SOD123_DIO"
 			(at 53.34 92.71 0)
 			(effects
@@
 			)
 		)
-		(property "Footprint" "JLCPCB:R_0402"
+		(property "Footprint" "footprints:R_0402"
 			(at 139.954 132.334 90)
 			(effects
@@
 			)
 		)
-		(property "Footprint" "JLCPCB:R_0402"
+		(property "Footprint" "footprints:R_0402"
 			(at 157.734 85.344 90)
 			(effects
@@
 			)
 		)
-		(property "Footprint" "JLCPCB:R_0402"
+		(property "Footprint" "footprints:R_0402"
 			(at 226.314 58.166 90)
 			(effects
@@
 			)
 		)
-		(property "Footprint" "BZT52C5V1_7_F:SOD123_DIO"
+		(property "Footprint" "footprints:SOD123_DIO"
 			(at 45.72 44.45 0)
 			(effects
@@
 			)
 		)
-		(property "Footprint" "SMLVN6RBG1U1:LED_SMLV56_ROM"
+		(property "Footprint" "footprints:LED_SMLV56_ROM"
 			(at 171.45 39.37 0)
 			(effects
@@
 			)
 		)
-		(property "Footprint" "JLCPCB:R_0402"
+		(property "Footprint" "footprints:R_0402"
 			(at 29.464 28.194 90)
 			(effects
@@
 			)
 		)
-		(property "Footprint" "BZT52C5V1_7_F:SOD123_DIO"
+		(property "Footprint" "footprints:SOD123_DIO"
 			(at 90.17 92.71 0)
 			(effects

Commit message: spdif fpga bansks
Parts:
- removed SW2, SW3, SW4, SW5: SW_Push, symbol Switch:SW_Push
- removed SW6, SW7: SW_SP3T, symbol Switch2:SW_SP3T
- added S3, S4, S5, S6: PTS645SK50SMTR92LFS, footprints:SW_PTS645SK50SMTR92LFS, symbol PTS645SK50SMTR92LFS:PTS645SK50SMTR92LFS
- added SW1, SW2: SW_SPDT, footprints:SS-12D10G5_XKB, symbol Switch2:SW_SPDT
- P1, P2: footprint pmod-conn_6x2:pmod_pin_array_6x2 -> footprints:CONN_PPPC062LJBN-RC_SUL
Connections:
- net +3.3V: now also S3.1, S4.1, S5.1, S6.1, SW1.3 (C), SW2.3 (C)
- net GNDREF: now also SW1.1 (A), SW2.1 (A)
- net at R15.1, R27.1: now also S6.3
- net at R21.1, R26.1: now also S5.3
- net at R22.1, R25.1: now also S4.3
- net at R29.1: now also SW2.2 (B)
- net at R23.1, R24.1: now also S3.3
- net at R28.1: now also SW1.2 (B)

Commit message: All pages complete , pi header left
Parts:
- removed S3, S4, S5, S6: PTS645SK50SMTR92LFS, footprints:SW_PTS645SK50SMTR92LFS, symbol PTS645SK50SMTR92LFS:PTS645SK50SMTR92LFS
- added S6, S7, S8, S9: PTS645SK50SMTR92LFS, footprints:SW_PTS645SK50SMTR92LFS, symbol PTS645SK50SMTR92LFS_:PTS645SK50SMTR92LFS
Connections:
- net +3.3V: now also S6.1, S7.1, S8.1, S9.1
- net GNDREF: now also D11.2 (A), D9.2 (A)
- net at R15.1, R27.1: now also S7.3
- net JA4_P: now reaches R77.1
- net JA4_N: now reaches R78.1
- net JA3_N: now reaches R76.1
- net JA1_P: now reaches R67.1
- net JB1_P: now reaches R71.1
- net at R22.1, R25.1: now also S8.3
- net JA2_P: now reaches R69.1
- net at R21.1, R26.1: now also S6.3
- net at R23.1, R24.1: now also S9.3
- net JA2_N: now reaches R70.1
- net JB2_P: now reaches R73.1
- net JB4_N: now reaches R82.1
- net JB3_P: now reaches R79.1
- net JB4_P: now reaches R81.1
- net JB1_N: now reaches R72.1
- net JB2_N: now reaches R74.1
- net JA3_P: now reaches R75.1
- net JB3_N: now reaches R80.1
- net JA1_N: now reaches R68.1

Commit message: update
Parts:
- D1, D4, D5, D6: footprint LED_SMD:LED_0402_1005Metric -> footprints:LED_0402_1005Metric
- Q1, Q2, Q3, Q4, Q5, Q6: footprint Package_TO_SOT_THT:TO-18-3 -> footprints:TO-18-3
Connections:
- net led0 renamed LED0
- net led1 renamed LED1
- net led2 renamed LED2
- net led3 renamed LED3
Changed lines of the file:
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@@
 		)
 	)
-	(global_label "led2"
+	(global_label "LED2"
 		(shape output)
 		(at 29.21 147.32 180)
@@
 		)
 		(property "Intersheetrefs" "${INTERSHEET_REFS}"
-			(at 22.1125 147.32 0)
+			(at 21.5682 147.32 0)
 			(effects
 				(font
@@
 		)
 	)
-	(global_label "led0"
+	(global_label "LED0"
 		(shape output)
 		(at 29.21 170.18 180)
@@
 		)
 		(property "Intersheetrefs" "${INTERSHEET_REFS}"
-			(at 22.1125 170.18 0)
+			(at 21.5682 170.18 0)
 			(effects
 				(font
@@
 		)
 	)
-	(global_label "led1"
+	(global_label "LED1"
 		(shape output)
 		(at 29.21 158.75 180)
@@
 		)
 		(property "Intersheetrefs" "${INTERSHEET_REFS}"
-			(at 22.1125 158.75 0)
+			(at 21.5682 158.75 0)
 			(effects
 				(font
@@
 		)
 	)
-	(global_label "led3"
+	(global_label "LED3"
 		(shape output)
 		(at 29.21 135.89 180)
@@
 		)
 		(property "Intersheetrefs" "${INTERSHEET_REFS}"
-			(at 22.1125 135.89 0)
+			(at 21.5682 135.89 0)
 			(effects
 				(font
@@
 			)
 		)
-		(property "Footprint" "Package_TO_SOT_THT:TO-18-3"
+		(property "Footprint" "footprints:TO-18-3"
 			(at 182.88 52.705 0)
 			(effects
@@
 			)
 		)
-		(property "Footprint" "LED_SMD:LED_0402_1005Metric"
+		(property "Footprint" "footprints:LED_0402_1005Metric"
 			(at 48.26 147.32 0)
 			(effects
@@
 			)
 		)
-		(property "Footprint" "LED_SMD:LED_0402_1005Metric"
+		(property "Footprint" "footprints:LED_0402_1005Metric"
 			(at 48.26 135.89 0)
 			(effects
@@
 			)
 		)
-		(property "Footprint" "Package_TO_SOT_THT:TO-18-3"
+		(property "Footprint" "footprints:TO-18-3"
 			(at 182.88 103.505 0)
 			(effects
@@
 			)
 		)
-		(property "Footprint" "Package_TO_SOT_THT:TO-18-3"
+		(property "Footprint" "footprints:TO-18-3"
 			(at 182.88 88.265 0)
 			(effects
@@
 			)
 		)
-		(property "Footprint" "Package_TO_SOT_THT:TO-18-3"
+		(property "Footprint" "footprints:TO-18-3"
 			(at 182.88 37.465 0)
 			(effects
@@
 			)
 		)
-		(property "Footprint" "LED_SMD:LED_0402_1005Metric"
+		(property "Footprint" "footprints:LED_0402_1005Metric"
 			(at 48.26 170.18 0)
 			(effects
@@
 			)
 		)
-		(property "Footprint" "LED_SMD:LED_0402_1005Metric"
+		(property "Footprint" "footprints:LED_0402_1005Metric"
 			(at 48.26 158.75 0)
 			(effects
@@
 			)
 		)
-		(property "Footprint" "Package_TO_SOT_THT:TO-18-3"
+		(property "Footprint" "footprints:TO-18-3"
 			(at 182.88 73.025 0)
 			(effects
@@
 			)
 		)
-		(property "Footprint" "Package_TO_SOT_THT:TO-18-3"
+		(property "Footprint" "footprints:TO-18-3"
 			(at 182.88 22.225 0)
 			(effects
