File: FPGA-BOARDver3/SPDIF.kicad_sch (KiCad schematic)
At the start: 6 parts, among them U5 TOTX1950AF, U6 TORX1950AF

Commit message: updated schematic and layout
Parts:
- C10, C11: LCSC PN (none) -> c1525
- L1: footprint footprints:L_0402 -> footprints:IND_TAIYO_CBC2012_TAY; LCSC PN (none) -> C223186
- R52: LCSC PN (none) -> C163457
- U5, U6: LCSC PN (none) -> mouser
Changed lines of the file:
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@@
 			)
 		)
-		(property "lcsc#" ""
+		(property "LCSC PN" "mouser"
 			(at 128.27 58.42 0)
 			(effects
@@
 			)
 		)
-		(property "lcsc#" ""
+		(property "LCSC PN" "mouser"
 			(at 133.35 110.49 0)
 			(effects
@@
 			)
 		)
-		(property "lcsc#" ""
+		(property "LCSC PN" "c1525"
 			(at 119.38 60.96 0)
 			(effects
@@
 			)
 		)
-		(property "lcsc#" ""
+		(property "LCSC PN" "c1525"
 			(at 120.65 115.57 0)
 			(effects
@@
 			)
 		)
-		(property "Footprint" "footprints:L_0402"
+		(property "Footprint" "footprints:IND_TAIYO_CBC2012_TAY"
 			(at 127 117.602 90)
 			(effects
@@
 			)
 		)
-		(property "lcsc#" ""
+		(property "LCSC PN" "C223186"
 			(at 127 119.38 0)
 			(effects
@@
 			)
 		)
-		(property "lcsc#" ""
+		(property "LCSC PN" "C163457"
 			(at 125.73 62.23 0)
 			(effects
