File: DDR and MIO banks.kicad_sch (KiCad schematic)
At the start: 42 parts, among them J4 Conn_01x04_Pin, J5 Conn_01x02_Pin, J8 Conn_01x02_Pin, U1 XC7Z020-1CLG400I__, U23 NC7WZ07P6X, Y2 SG-8018CE_50.0000M-TJHPA

Commit message: ready for manufacturing
Parts:
- BTNR1: LCSC PN mouser -> C221872
- C176, C4: footprint footprints:C_0402 -> footprints:C_0201_0603Metric; LCSC PN c1525 -> c307380
- C5: footprint footprints:C_0402 -> footprints:C_0201_0603Metric; LCSC PN c15195 -> c85930
- C8: LCSC PN c15195 -> c85930
- C9: footprint footprints:C_0402 -> footprints:C_0201_0603Metric; LCSC PN c15195 -> c307380
- J4, J5, J8: LCSC PN digi/mouser -> (none)
- R234, R235, R236, R237, R238, R239, R4: value 40.2 -> 40.2 1%
- R36, R37, R38, R40, R42, R48, R49: value 20K -> 20K 1%
- R43, R45: value 10K -> 10K 1%
- R5: LCSC PN C843839 -> C106232
Connections:
- net DDR3_D1: now also U1.G3 (PS_DDR_DQ10_502); no longer U1.H1 (PS_DDR_DQ14_502)
- net DDR3_D11: now also U1.A2 (PS_DDR_DQ2_502); no longer U1.C1 (PS_DDR_DQ6_502)
- net DDR3_D12: now also U1.C1 (PS_DDR_DQ6_502); no longer U1.B3 (PS_DDR_DQ1_502)
- net DDR3_D14: now also U1.D1 (PS_DDR_DQ5_502); no longer U1.C3 (PS_DDR_DQ0_502)
- net DDR3_D15: now also U1.B3 (PS_DDR_DQ1_502); no longer U1.A2 (PS_DDR_DQ2_502)
- net DDR3_D3: now also U1.H1 (PS_DDR_DQ14_502); no longer U1.G3 (PS_DDR_DQ10_502)
- net DDR3_D4: now also U1.H3 (PS_DDR_DQ11_502); no longer U1.J1 (PS_DDR_DQ15_502)
- net DDR3_D5: now also U1.J1 (PS_DDR_DQ15_502); no longer U1.H3 (PS_DDR_DQ11_502)
- net DDR3_D9: now also U1.C3 (PS_DDR_DQ0_502); no longer U1.D1 (PS_DDR_DQ5_502)
