File: DDR and MIO banks.kicad_sch (KiCad schematic)
At the start: 42 parts, among them J4 Conn_01x04_Pin, J5 Conn_01x02_Pin, J8 Conn_01x02_Pin, U1 XC7Z020-1CLG400I__, U23 NC7WZ07P6X, Y2 SG-8018CE_50.0000M-TJHPA

Commit message: post -production rework
Connections:
- net +3V3: now also J8.2 (Pin_2)
- net UART_RXD renamed UART_RXD_OUT
- net UART_TXD renamed UART_TXD_IN
