File: FPGA_POWER.kicad_sch (KiCad schematic)
At the start: 56 parts, among them U1 XC7Z020-1CLG400I__

Commit message: new layout by abdul
Parts:
- C100, C101, C102, C103, C104, C105, C106, C107, C108, C109, C110, C111, C112, C113, C87, C88, C89, C90, C91, C92, C93, C94, C95, C96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: footprint footprints:C_0402 -> footprints:C_0201_0603Metric; LCSC PN c92361 -> C88915
Other:
- moved on the sheet: C100, C101, C102, C103
