File: FPGA_POWER.kicad_sch (KiCad schematic)
At the start: 56 parts, among them U1 XC7Z020-1CLG400I__

Commit message: ready for manufacturing
Parts:
- C100, C101, C102, C103, C104, C105, C106, C107, C108, C109, C110, C111, C112, C113, C87, C88, C89, C90, C91, C92, C93, C94, C95, C96, C97, C98, C99: LCSC PN C88915 -> C5383023
- C114, C115, C117, C118, C119, C120, C121, C122, C123, C124, C126, C127, C86: LCSC PN c23733 -> C2858031
- C125, C138: LCSC PN c16790 -> C124129
- C137: value 10uF -> 10uF 10V; footprint footprints:C_0402 -> footprints:C_0805; LCSC PN c315248 -> C15850
- FL1: value 600Ohm/100MHz -> 600Ohm/100Mhz; LCSC PN digi/mouser -> C19330
