File: JTAG.kicad_sch (KiCad schematic)
At the start: 21 parts, among them U1 XC7Z020-1CLG400I__, U4 ATSHA204A-SSHCZ-T, U7 S25FL128SAGMFI000

Commit message: new layout by abdul
Parts:
- C12, C13, C15, C16: footprint footprints:C_0402 -> footprints:C_0201_0603Metric
Other:
- moved on the sheet: C13
Changed lines of the file:
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@@
 	)
 	(junction
-		(at 175.26 119.38)
+		(at 50.8 135.89)
 		(diameter 0)
 		(color 0 0 0 0)
 	)
 	(junction
-		(at 251.46 91.44)
+		(at 175.26 119.38)
 		(diameter 0)
 		(color 0 0 0 0)
 	)
 	(junction
-		(at 250.19 69.85)
+		(at 251.46 91.44)
 		(diameter 0)
 		(color 0 0 0 0)
 	)
 	(junction
-		(at 127 138.43)
+		(at 250.19 69.85)
 		(diameter 0)
 		(color 0 0 0 0)
 	)
 	(junction
-		(at 49.53 135.89)
+		(at 127 138.43)
 		(diameter 0)
 		(color 0 0 0 0)
 	)
 	(junction
-		(at 49.53 144.78)
+		(at 267.97 91.44)
 		(diameter 0)
 		(color 0 0 0 0)
 	)
 	(junction
-		(at 267.97 91.44)
+		(at 50.8 144.78)
 		(diameter 0)
 		(color 0 0 0 0)
@@
 	(wire
 		(pts
+			(xy 50.8 144.78) (xy 60.96 144.78)
+		)
+		(stroke
+			(width 0)
+			(type default)
+		)
+	)
+	(wire
+		(pts
 			(xy 60.96 140.97) (xy 60.96 144.78)
 		)
@@
 	(wire
 		(pts
-			(xy 45.72 135.89) (xy 49.53 135.89)
+			(xy 45.72 135.89) (xy 50.8 135.89)
 		)
 		(stroke
@@
 	(wire
 		(pts
-			(xy 60.96 135.89) (xy 49.53 135.89)
+			(xy 60.96 135.89) (xy 50.8 135.89)
 		)
 		(stroke
@@
 	(wire
 		(pts
-			(xy 138.43 36.83) (xy 149.86 36.83)
+			(xy 50.8 137.16) (xy 50.8 135.89)
 		)
 		(stroke
@@
 	(wire
 		(pts
-			(xy 124.46 121.92) (xy 142.24 121.92)
+			(xy 138.43 36.83) (xy 149.86 36.83)
 		)
 		(stroke
@@
 	(wire
 		(pts
-			(xy 124.46 140.97) (xy 127 140.97)
+			(xy 124.46 121.92) (xy 142.24 121.92)
 		)
 		(stroke
@@
 	(wire
 		(pts
-			(xy 142.24 34.29) (xy 153.67 34.29)
+			(xy 124.46 140.97) (xy 127 140.97)
 		)
 		(stroke
@@
 	(wire
 		(pts
-			(xy 175.26 119.38) (xy 175.26 120.65)
+			(xy 142.24 34.29) (xy 153.67 34.29)
 		)
 		(stroke
@@
 	(wire
 		(pts
-			(xy 196.85 69.85) (xy 219.71 69.85)
+			(xy 175.26 119.38) (xy 175.26 120.65)
 		)
 		(stroke
@@
 	(wire
 		(pts
-			(xy 49.53 144.78) (xy 49.53 143.51)
+			(xy 196.85 69.85) (xy 219.71 69.85)
 		)
 		(stroke
@@
 	(wire
 		(pts
-			(xy 45.72 144.78) (xy 49.53 144.78)
+			(xy 45.72 144.78) (xy 50.8 144.78)
 		)
 		(stroke
@@
 	(wire
 		(pts
-			(xy 49.53 144.78) (xy 60.96 144.78)
-		)
-		(stroke
-			(width 0)
-			(type default)
-		)
-	)
-	(wire
-		(pts
 			(xy 251.46 91.44) (xy 267.97 91.44)
 		)
@@
 			)
 		)
-		(property "Footprint" "footprints:C_0402"
+		(property "Footprint" "footprints:C_0201_0603Metric"
 			(at 197.8152 77.47 0)
 			(effects
@@
 	(symbol
 		(lib_id "Device:C")
-		(at 49.53 139.7 0)
+		(at 50.8 140.97 0)
 		(unit 1)
 		(exclude_from_sim no)
@@
 		(fields_autoplaced yes)
 		(property "Reference" "C13"
-			(at 53.34 138.4299 0)
+			(at 54.61 139.6999 0)
 			(effects
 				(font
@@
 		)
 		(property "Value" "100nF"
-			(at 53.34 140.9699 0)
+			(at 54.61 142.2399 0)
 			(effects
 				(font
@@
 			)
 		)
-		(property "Footprint" "footprints:C_0402"
-			(at 50.4952 143.51 0)
+		(property "Footprint" "footprints:C_0201_0603Metric"
+			(at 51.7652 144.78 0)
 			(effects
 				(font
@@
 		)
 		(property "Datasheet" "~"
-			(at 49.53 139.7 0)
+			(at 50.8 140.97 0)
 			(effects
 				(font
@@
 		)
 		(property "Description" "Unpolarized capacitor"
-			(at 49.53 139.7 0)
+			(at 50.8 140.97 0)
 			(effects
 				(font
@@
 		)
 		(property "LCSC PN" "c1525"
-			(at 49.53 139.7 0)
+			(at 50.8 140.97 0)
 			(effects
 				(font
@@
 			)
 		)
-		(property "Footprint" "footprints:C_0402"
+		(property "Footprint" "footprints:C_0201_0603Metric"
 			(at 35.2552 129.54 0)
 			(effects
@@
 			)
 		)
-		(property "Footprint" "footprints:C_0402"
+		(property "Footprint" "footprints:C_0201_0603Metric"
 			(at 49.2252 116.84 0)
 			(effects
@@
 		(lib_id "Device:R_US")
 		(at 175.26 124.46 0)
+		(mirror y)
 		(unit 1)
 		(exclude_from_sim no)
@@
 		(on_board yes)
 		(dnp no)
-		(fields_autoplaced yes)
 		(property "Reference" "R115"
-			(at 177.8 123.1899 0)
+			(at 172.72 123.1899 0)
 			(effects
 				(font
@@
 		)
 		(property "Value" "220"
-			(at 177.8 125.7299 0)
+			(at 172.72 125.7299 0)
 			(effects
 				(font
@@
 		)
 		(property "Footprint" "footprints:R_0402"
-			(at 176.276 124.714 90)
+			(at 174.244 124.714 90)
 			(effects
 				(font

Commit message: Layout update
Parts:
- added C206: 100nF, footprints:C_0201_0603Metric, symbol Device:C
- added J7: JTAG Header, footprints:PinHeader_1x06_P2.54mm_Vertical, symbol Connector:Conn_01x06_Pin
- added RV3, RV4, RV5, RV6: CG0402MLU-3.3G, footprints:VARC1005X41N, symbol CG0402MLU-3_3G:CG0402MLU-3.3G
- R118, R119, R120, R121: value 100 -> 22; footprint footprints:R_0402 -> footprints:R_0201_0603Metric; LCSC PN C106232 -> (none)
Connections:
- net +3V3: now also C206.1, J7.6 (VDD)
- net GNDREF: now also U7.3 (RESET#/RFU), C206.2, J7.5 (GND), RV3.2, RV4.2, RV5.2, RV6.2
- net TCK: now also R120.1, U1.F9 (TCK_0); no longer R120.2
- net TDI: now also R118.1, U1.G6 (TDI_0); no longer R119.2
- net TDO: now also R119.1, U1.F6 (TDO_0); no longer R121.2
- net TMS: now also R121.1, U1.J6 (TMS_0); no longer R118.2
- new net JTAG_TCK: J7.4 (TCK), R120.2, RV5.1
- new net JTAG_TDI: J7.2 (TDI), R118.2, RV3.1
- new net JTAG_TDO: J7.3 (TDO), R119.2, RV4.1
- new net JTAG_TMS: J7.1 (TMS), R121.2, RV6.1
Other:
- moved on the sheet: C12, C13, C14, C15, C16, DONE1, R114, R115, R116, R117, R122, R123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
