File: JTAG.kicad_sch (KiCad schematic)
At the start: 27 parts, among them J7 JTAG Header, U1 XC7Z020-1CLG400I__, U10 TPD1E05U06DPYR, U37 TPD1E05U06DPYR, U38 TPD1E05U06DPYR, U39 TPD1E05U06DPYR, U4 ATSHA204A-SSHCZ-T, U7 S25FL128SAGMFI000

Commit message: post -production rework
Parts:
- removed DONE1: Green, footprints:LED_0402_1005Metric, symbol Aquiot:LED
- removed U7: S25FL128SAGMFI000, footprints:SO3016_INF, symbol S25FL128SAGMFI000:S25FL128SAGMFI000
- added D9: LED, footprints:LED_0402_1005Metric, symbol Device:LED
- added U17: W25Q128JVSIQ, footprints:SOIC127P790X216-8N, symbol W25Q128JVSIQ:W25Q128JVSIQ
- C15, R117, U4: now left out of the parts list
Connections:
- net +3V3: now also U17.8 (VCC)
- net GNDREF: now also D9.1 (K), U17.4 (GND)
- net SPI_CS: now also U17.1 (/CS)
- net SPI_DQ0/MODE3: now also U17.5 (DI(IO0))
- net SPI_DQ1/MODE1: now also U17.2 (DO(IO1))
- net SPI_DQ2/MODE2: now also U17.3 (/WP(IO2))
- net SPI_DQ3/MODE0: now also U17.7 (/HOLD/RESET(IO3))
- net SPI_SCK/MODE4: now also U17.6 (CLK)
- net at R115.2: now also D9.2 (A)
