File: USB_JTAG_PROGRAMMING.kicad_sch (KiCad schematic)
At the start: 46 parts, among them J16 10118194-0001LF, U15 93LC56B-I/SN, U3 FT2232HQ, U34 TPD1E05U06DPYR, U35 TPD1E05U06DPYR, Y3 SIT1602AC-12-33E-12.000000G

Commit message: post -production rework
Parts:
- removed led_rx1, led_tx1: Green, footprints:LED_0402_1005Metric, symbol Aquiot:LED
- added D10, D11: LED, footprints:LED_0402_1005Metric, symbol Device:LED
- R205, R208: LCSC PN C713499 -> C18164337
Connections:
- net +3V3: now also U3.21 (ADBUS4)
- net FTDI_RX_LED_K: now also D10.1 (K)
- net at R205.1: now also D10.2 (A)
- net at R112.1: now also U3.23 (ADBUS6); no longer U3.22 (ADBUS5)
- net at R208.1: now also D11.2 (A)
- net FTDI_TX_KED_K renamed FTDI_TX_LED_K
- net FTDI_TX_LED_K: now also D11.1 (K)
- net UART_RXD renamed UART_TXD_IN
- net UART_TXD renamed UART_RXD_OUT
Other:
- moved on the sheet: C201, R111, R112, R209, R210, R51
