File: AUDIO.kicad_sch (KiCad schematic)
At the start: 47 parts, among them J15 USB-A-S-X-X-SM2, J9 SJ1-3525NG, Q10 DMG2305UX-13, U10 AD8647ARMZ-REEL, U21 NC7WZ07P6X, U25 TPS2051BDBVR, U26 TUSB1210BRHBT, U35 TPD4E05U06DQAR

Commit message: update
Parts:
- added R204: 0, footprints:R_0402, symbol Device:R_US
Connections:
- net VCC1V8_IO: now also R204.2; no longer C190.2, C191.2, U26.28 (VDD18), U26.30 (VDD18)
- new net: C190.2, C191.2, R204.1, U26.28 (VDD18), U26.30 (VDD18)
Other:
- moved on the sheet: C182
Changed lines of the file:
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@@
 	(wire
 		(pts
+			(xy 180.34 20.32) (xy 184.15 20.32)
+		)
+		(stroke
+			(width 0)
+			(type default)
+		)
+	)
+	(wire
+		(pts
 			(xy 160.02 95.25) (xy 171.45 95.25)
 		)
@@
 	(wire
 		(pts
-			(xy 168.91 20.32) (xy 184.15 20.32)
+			(xy 168.91 20.32) (xy 172.72 20.32)
 		)
 		(stroke
@@
 	(symbol
 		(lib_id "Device:C")
-		(at 83.82 90.17 0)
-		(mirror x)
+		(at 83.82 90.17 180)
 		(unit 1)
 		(exclude_from_sim no)
@@
 		(dnp no)
 		(property "Reference" "C182"
-			(at 83.566 90.424 0)
+			(at 84.074 90.424 0)
 			(effects
 				(font
@@
 		)
 		(property "Value" "1uF 10V"
-			(at 86.106 92.456 0)
+			(at 81.534 92.456 0)
 			(effects
 				(font
@@
 		)
 		(property "Footprint" "footprints:C_0402"
-			(at 84.7852 86.36 0)
+			(at 82.8548 86.36 0)
 			(effects
 				(font
@@
 	)
 	(symbol
+		(lib_id "Device:R_US")
+		(at 176.53 20.32 270)
+		(unit 1)
+		(exclude_from_sim no)
+		(in_bom yes)
+		(on_board yes)
+		(dnp no)
+		(property "Reference" "R204"
+			(at 178.308 14.224 0)
+			(effects
+				(font
+					(size 1.27 1.27)
+				)
+				(justify left)
+			)
+		)
+		(property "Value" "0"
+			(at 175.768 15.748 0)
+			(effects
+				(font
+					(size 1.27 1.27)
+				)
+				(justify left)
+			)
+		)
+		(property "Footprint" "footprints:R_0402"
+			(at 176.276 21.336 90)
+			(effects
+				(font
+					(size 1.27 1.27)
+				)
+				(hide yes)
+			)
+		)
+		(property "Datasheet" "~"
+			(at 176.53 20.32 0)
+			(effects
+				(font
+					(size 1.27 1.27)
+				)
+				(hide yes)
+			)
+		)
+		(property "Description" "Resistor, US symbol"
+			(at 176.53 20.32 0)
+			(effects
+				(font
+					(size 1.27 1.27)
+				)
+				(hide yes)
+			)
+		)
+		(property "LCSC PN" "C106231"
+			(at 176.53 20.32 0)
+			(effects
+				(font
+					(size 1.27 1.27)
+				)
+				(hide yes)
+			)
+		)
+		(pin "1"
+		)
+		(pin "2"
+		)
+		(instances
+			(project "FPGA-BOARDver3"
+				(path "/4a327bdf-04e5-4836-9c0a-5fb801c23f64/cd0c3344-baf7-4bb5-a300-e73c15154941"
+					(reference "R204")
+					(unit 1)
+				)
+			)
+		)
+	)
+	(symbol
 		(lib_id "power:GNDREF")
 		(at 234.95 48.26 90)
@@
 		(lib_id "Device:R_US")
 		(at 76.2 90.17 0)
-		(mirror y)
 		(unit 1)
 		(exclude_from_sim no)
@@
 		(dnp no)
 		(property "Reference" "R200"
-			(at 75.184 88.646 0)
+			(at 77.216 88.646 0)
 			(effects
 				(font
@@
 		)
 		(property "Value" "0"
-			(at 74.676 91.186 0)
+			(at 77.724 91.186 0)
 			(effects
 				(font
@@
 		)
 		(property "Footprint" "footprints:R_0402"
-			(at 75.184 90.424 90)
+			(at 77.216 90.424 90)
 			(effects
 				(font
