File: AUDIO.kicad_sch (KiCad schematic)
At the start: 49 parts, among them J15 USB-A-S-X-X-SM2, J9 SJ1-3525NG, Q10 DMG2305UX-13, U10 AD8647ARMZ-REEL, U21 NC7WZ07P6X, U25 TPS2051BDBVR, U26 TUSB1210BRHBT, U35 TPD4E05U06DQAR

Commit message: new layout by abdul
Parts:
- removed R205: 0, footprints:R_0402, symbol Device:R_US
- C1, C189, C190, C191, C2: footprint footprints:C_0402 -> footprints:C_0201_0603Metric
Connections:
- net +5V: no longer R202.2, U25.4 (EN), U26.17 (CPEN)
- net GNDREF: no longer U35.3 (GND)
- new net: R202.2, U25.4 (EN), U26.17 (CPEN)
Other:
- moved on the sheet: R193, U35
Changed lines of the file:
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@@
 	(paper "A4")
 	(junction
-		(at 104.14 71.12)
-		(diameter 0)
-		(color 0 0 0 0)
-	)
-	(junction
-		(at 171.45 83.82)
-		(diameter 0)
-		(color 0 0 0 0)
-	)
-	(junction
 		(at 165.1 143.51)
 		(diameter 0)
@@
 	)
 	(junction
-		(at 160.02 83.82)
-		(diameter 0)
-		(color 0 0 0 0)
-	)
-	(junction
 		(at 102.87 129.54)
 		(diameter 0)
@@
 	)
 	(junction
-		(at 184.15 27.94)
-		(diameter 0)
-		(color 0 0 0 0)
-	)
-	(junction
 		(at 109.22 59.69)
 		(diameter 0)
@@
 	)
 	(junction
-		(at 109.22 71.12)
+		(at 171.45 73.66)
 		(diameter 0)
 		(color 0 0 0 0)
@@
 	(wire
 		(pts
+			(xy 157.48 73.66) (xy 171.45 73.66)
+		)
+		(stroke
+			(width 0)
+			(type default)
+		)
+	)
+	(wire
+		(pts
 			(xy 57.15 115.57) (xy 57.15 113.03)
 		)
@@
 	(wire
 		(pts
-			(xy 104.14 71.12) (xy 109.22 71.12)
-		)
-		(stroke
-			(width 0)
-			(type default)
-		)
-	)
-	(wire
-		(pts
 			(xy 15.24 58.42) (xy 15.24 72.39)
 		)
@@
 	(wire
 		(pts
-			(xy 171.45 83.82) (xy 171.45 86.36)
-		)
-		(stroke
-			(width 0)
-			(type default)
-		)
-	)
-	(wire
-		(pts
 			(xy 72.39 140.97) (xy 82.55 140.97)
 		)
@@
 	(wire
 		(pts
-			(xy 160.02 83.82) (xy 171.45 83.82)
+			(xy 205.74 107.95) (xy 208.28 107.95)
 		)
 		(stroke
@@
 	(wire
 		(pts
-			(xy 205.74 107.95) (xy 208.28 107.95)
+			(xy 171.45 93.98) (xy 171.45 95.25)
 		)
 		(stroke
@@
 	(wire
 		(pts
-			(xy 171.45 93.98) (xy 171.45 95.25)
+			(xy 100.33 142.24) (xy 102.87 142.24)
 		)
 		(stroke
@@
 	(wire
 		(pts
-			(xy 100.33 142.24) (xy 102.87 142.24)
+			(xy 207.01 27.94) (xy 204.47 27.94)
 		)
 		(stroke
@@
 	(wire
 		(pts
-			(xy 207.01 27.94) (xy 204.47 27.94)
+			(xy 76.2 85.09) (xy 68.58 85.09)
 		)
 		(stroke
@@
 	(wire
 		(pts
-			(xy 76.2 85.09) (xy 68.58 85.09)
+			(xy 157.48 83.82) (xy 157.48 73.66)
 		)
 		(stroke
@@
 	(wire
 		(pts
-			(xy 168.91 27.94) (xy 172.72 27.94)
-		)
-		(stroke
-			(width 0)
-			(type default)
-		)
-	)
-	(wire
-		(pts
 			(xy 43.18 57.15) (xy 91.44 57.15)
 		)
@@
 	(wire
 		(pts
-			(xy 154.94 83.82) (xy 160.02 83.82)
-		)
-		(stroke
-			(width 0)
-			(type default)
-		)
-	)
-	(wire
-		(pts
 			(xy 66.04 85.09) (xy 68.58 85.09)
 		)
@@
 	(wire
 		(pts
+			(xy 154.94 83.82) (xy 157.48 83.82)
+		)
+		(stroke
+			(width 0)
+			(type default)
+		)
+	)
+	(wire
+		(pts
 			(xy 57.15 123.19) (xy 57.15 129.54)
 		)
@@
 	(wire
 		(pts
-			(xy 184.15 27.94) (xy 180.34 27.94)
+			(xy 243.84 134.62) (xy 251.46 134.62)
 		)
 		(stroke
@@
 	(wire
 		(pts
-			(xy 243.84 134.62) (xy 251.46 134.62)
+			(xy 83.82 97.79) (xy 76.2 97.79)
 		)
 		(stroke
@@
 	(wire
 		(pts
-			(xy 83.82 97.79) (xy 76.2 97.79)
+			(xy 67.31 71.12) (xy 66.04 71.12)
 		)
 		(stroke
@@
 	(wire
 		(pts
-			(xy 67.31 71.12) (xy 66.04 71.12)
+			(xy 66.04 59.69) (xy 95.25 59.69)
 		)
 		(stroke
@@
 	(wire
 		(pts
-			(xy 66.04 59.69) (xy 95.25 59.69)
+			(xy 118.11 129.54) (xy 115.57 129.54)
 		)
 		(stroke
@@
 	(wire
 		(pts
-			(xy 118.11 129.54) (xy 115.57 129.54)
+			(xy 229.87 90.17) (xy 231.14 90.17)
 		)
 		(stroke
@@
 	(wire
 		(pts
-			(xy 229.87 90.17) (xy 231.14 90.17)
+			(xy 171.45 73.66) (xy 171.45 86.36)
 		)
 		(stroke
@@
 	(wire
 		(pts
-			(xy 171.45 83.82) (xy 171.45 64.77)
+			(xy 171.45 64.77) (xy 171.45 73.66)
 		)
 		(stroke
@@
 	)
 	(symbol
-		(lib_id "power:+1V8")
-		(at 168.91 27.94 90)
-		(unit 1)
-		(exclude_from_sim no)
-		(in_bom yes)
-		(on_board yes)
-		(dnp no)
-		(fields_autoplaced yes)
-		(property "Reference" "#PWR0261"
-			(at 172.72 27.94 0)
-			(effects
-				(font
-					(size 1.27 1.27)
-				)
-				(hide yes)
-			)
-		)
-		(property "Value" "+1V8"
-			(at 165.1 27.9399 90)
-			(effects
-				(font
-					(size 1.27 1.27)
-				)
-				(justify left)
-			)
-		)
-		(property "Footprint" ""
-			(at 168.91 27.94 0)
-			(effects
-				(font
-					(size 1.27 1.27)
-				)
-				(hide yes)
-			)
-		)
-		(property "Datasheet" ""
-			(at 168.91 27.94 0)
-			(effects
-				(font
-					(size 1.27 1.27)
-				)
-				(hide yes)
-			)
-		)
-		(property "Description" "Power symbol creates a global label with name \"+1V8\""
-			(at 168.91 27.94 0)
-			(effects
-				(font
-					(size 1.27 1.27)
-				)
-				(hide yes)
-			)
-		)
-		(pin "1"
-		)
-		(instances
-			(project ""
-				(path "/4a327bdf-04e5-4836-9c0a-5fb801c23f64/cd0c3344-baf7-4bb5-a300-e73c15154941"
-					(reference "#PWR0261")
-					(unit 1)
-				)
-			)
-		)
-	)
-	(symbol
 		(lib_id "Device:C")
 		(at 72.39 148.59 0)
@@
 			)
 		)
-		(property "Footprint" "footprints:C_0402"
+		(property "Footprint" "footprints:C_0201_0603Metric"
 			(at 254.9652 158.75 0)
 			(effects
@@
 			)
 		)
-		(property "Footprint" "footprints:C_0402"
+		(property "Footprint" "footprints:C_0201_0603Metric"
 			(at 197.1548 17.78 0)
 			(effects
@@
 			)
 		)
-		(property "Footprint" "footprints:C_0402"
+		(property "Footprint" "footprints:C_0201_0603Metric"
 			(at 252.4252 130.81 0)
 			(effects
@@
 	(symbol
 		(lib_id "Device:R_US")
-		(at 81.28 157.48 180)
+		(at 81.28 157.48 0)
+		(mirror x)
 		(unit 1)
 		(exclude_from_sim no)
@@
 		(dnp no)
 		(property "Reference" "R193"
-			(at 80.264 159.004 0)
+			(at 82.296 159.004 0)
 			(effects
 				(font
@@
 		)
 		(property "Value" "10K"
-			(at 79.756 156.464 0)
+			(at 82.804 156.464 0)
 			(effects
 				(font
@@
 		)
 		(property "Footprint" "footprints:R_0402"
-			(at 80.264 157.226 90)
+			(at 82.296 157.226 90)
 			(effects
 				(font
@@
 			)
 		)
-		(property "Footprint" "footprints:C_0402"
+		(property "Footprint" "footprints:C_0201_0603Metric"
 			(at 184.4548 29.21 0)
 			(effects
@@
 		)
 		(property "Value" "10.7K 1%"
-			(at 73.914 135.636 0)
+			(at 71.628 134.874 0)
 			(effects
 				(font
@@
 	)
 	(symbol
-		(lib_id "Device:R_US")
-		(at 176.53 27.94 270)
-		(unit 1)
-		(exclude_from_sim no)
-		(in_bom yes)
-		(on_board yes)
-		(dnp no)
-		(property "Reference" "R205"
-			(at 178.308 21.844 0)
-			(effects
-				(font
-					(size 1.27 1.27)
-				)
-				(justify left)
-			)
-		)
-		(property "Value" "0"
-			(at 175.768 23.368 0)
-			(effects
-				(font
-					(size 1.27 1.27)
-				)
-				(justify left)
-			)
-		)
-		(property "Footprint" "footprints:R_0402"
-			(at 176.276 28.956 90)
-			(effects
-				(font
-					(size 1.27 1.27)
-				)
-				(hide yes)
-			)
-		)
-		(property "Datasheet" "~"
-			(at 176.53 27.94 0)
-			(effects
-				(font
-					(size 1.27 1.27)
-				)
-				(hide yes)
-			)
-		)
-		(property "Description" "Resistor, US symbol"
-			(at 176.53 27.94 0)
-			(effects
-				(font
-					(size 1.27 1.27)
-				)
-				(hide yes)
-			)
-		)
-		(property "LCSC PN" "C106231"
-			(at 176.53 27.94 0)
-			(effects
-				(font
-					(size 1.27 1.27)
-				)
-				(hide yes)
-			)
-		)
-		(pin "1"
-		)
-		(pin "2"
-		)
-		(instances
-			(project "FPGA-BOARDver3"
-				(path "/4a327bdf-04e5-4836-9c0a-5fb801c23f64/cd0c3344-baf7-4bb5-a300-e73c15154941"
-					(reference "R205")
-					(unit 1)
-				)
-			)
-		)
-	)
-	(symbol
 		(lib_id "TP2S051BDBVR:TPS2051BDBVR")
 		(at 142.24 86.36 0)
@@
 			)
 		)
-		(property "Footprint" "footprints:C_0402"
+		(property "Footprint" "footprints:C_0201_0603Metric"
 			(at 192.0748 29.21 0)
 			(effects

Commit message: update
Parts:
- removed R204: 0, footprints:R_0402, symbol Device:R_US
Connections:
- net VCC1V8_IO: now also C190.2, C191.2, U26.28 (VDD18), U26.30 (VDD18)
Other:
- moved on the sheet: C182
Changed lines of the file:
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@@
 	(wire
 		(pts
-			(xy 180.34 20.32) (xy 184.15 20.32)
-		)
-		(stroke
-			(width 0)
-			(type default)
-		)
-	)
-	(wire
-		(pts
 			(xy 160.02 95.25) (xy 171.45 95.25)
 		)
@@
 	(wire
 		(pts
-			(xy 168.91 20.32) (xy 172.72 20.32)
+			(xy 168.91 20.32) (xy 184.15 20.32)
 		)
 		(stroke
@@
 	(symbol
 		(lib_id "Device:C")
-		(at 83.82 90.17 180)
+		(at 83.82 90.17 0)
+		(mirror x)
 		(unit 1)
 		(exclude_from_sim no)
@@
 		(dnp no)
 		(property "Reference" "C182"
-			(at 84.074 90.424 0)
+			(at 83.566 90.424 0)
 			(effects
 				(font
@@
 		)
 		(property "Value" "1uF 10V"
-			(at 81.534 92.456 0)
+			(at 86.106 92.456 0)
 			(effects
 				(font
@@
 		)
 		(property "Footprint" "footprints:C_0402"
-			(at 82.8548 86.36 0)
+			(at 84.7852 86.36 0)
 			(effects
 				(font
@@
 	)
 	(symbol
-		(lib_id "Device:R_US")
-		(at 176.53 20.32 270)
-		(unit 1)
-		(exclude_from_sim no)
-		(in_bom yes)
-		(on_board yes)
-		(dnp no)
-		(property "Reference" "R204"
-			(at 178.308 14.224 0)
-			(effects
-				(font
-					(size 1.27 1.27)
-				)
-				(justify left)
-			)
-		)
-		(property "Value" "0"
-			(at 175.768 15.748 0)
-			(effects
-				(font
-					(size 1.27 1.27)
-				)
-				(justify left)
-			)
-		)
-		(property "Footprint" "footprints:R_0402"
-			(at 176.276 21.336 90)
-			(effects
-				(font
-					(size 1.27 1.27)
-				)
-				(hide yes)
-			)
-		)
-		(property "Datasheet" "~"
-			(at 176.53 20.32 0)
-			(effects
-				(font
-					(size 1.27 1.27)
-				)
-				(hide yes)
-			)
-		)
-		(property "Description" "Resistor, US symbol"
-			(at 176.53 20.32 0)
-			(effects
-				(font
-					(size 1.27 1.27)
-				)
-				(hide yes)
-			)
-		)
-		(property "LCSC PN" "C106231"
-			(at 176.53 20.32 0)
-			(effects
-				(font
-					(size 1.27 1.27)
-				)
-				(hide yes)
-			)
-		)
-		(pin "1"
-		)
-		(pin "2"
-		)
-		(instances
-			(project "FPGA-BOARDver3"
-				(path "/4a327bdf-04e5-4836-9c0a-5fb801c23f64/cd0c3344-baf7-4bb5-a300-e73c15154941"
-					(reference "R204")
-					(unit 1)
-				)
-			)
-		)
-	)
-	(symbol
 		(lib_id "power:GNDREF")
 		(at 234.95 48.26 90)
@@
 		(lib_id "Device:R_US")
 		(at 76.2 90.17 0)
+		(mirror y)
 		(unit 1)
 		(exclude_from_sim no)
@@
 		(dnp no)
 		(property "Reference" "R200"
-			(at 77.216 88.646 0)
+			(at 75.184 88.646 0)
 			(effects
 				(font
@@
 		)
 		(property "Value" "0"
-			(at 77.724 91.186 0)
+			(at 74.676 91.186 0)
 			(effects
 				(font
@@
 		)
 		(property "Footprint" "footprints:R_0402"
-			(at 77.216 90.424 90)
+			(at 75.184 90.424 90)
 			(effects
 				(font

Commit message: ready for manufacturing
Parts:
- removed CR3: DDZ9699-7, footprints:ZDO_SOD123_DIO, symbol DDZ9699-7:DDZ9699-7
- removed CR5: 7M-26.000MAAJ-T, footprints:CRYSTAL_TXC_7M, symbol 7M_26_000MAAJ_T:7M-26.000MAAJ-T
- removed U10: AD8647ARMZ-REEL, footprints:RM_10_ADI, symbol AD8647ARMZ:AD8647ARMZ-REEL
- removed U35: TPD4E05U06DQAR, footprints:IC_TPD4E05U06DQAR, symbol TPD4E05U06DQAR:TPD4E05U06DQAR
- added CR3: BZT52C12-7-F, footprints:SOD123_DIO, symbol BZT52C12_7_F:BZT52C12-7-F
- added U30: TPD4E05U06DQAR, footprints:IC_TPD4E05U06DQAR, symbol TPD4E05U06DQAR:TPD4E05U06DQAR
- added U36: AD8592ARM, footprints:RM_10_ADI, symbol AD8592ARM:AD8592ARM
- added Y4: ABM8G-26.000MHZ-18-D2Y-T, footprints:CRYSTAL_ABM8G_ABR, symbol ABM8G_26_000MHZ_18_D2Y_T:ABM8G-26.000MHZ-18-D2Y-T
- C1, C189, C190, C191, C2: LCSC PN c1525 -> c307380
- C181: LCSC PN c14442 -> C77018
- C182: LCSC PN c14445 -> C52923
- C183, C186: LCSC PN c71687 -> C77020
- C184: footprint footprints:C_0402 -> footprints:C_0201_0603Metric; LCSC PN c15195 -> c85930
- C185: value 4.7uF 10V -> 4.7uF; LCSC PN c368809 -> C2858031
- C187: footprint footprints:C_0402 -> footprints:C_0201_0603Metric; LCSC PN c1525 -> c307380
- R193: value 10K -> 10K 1%
- R196: value 2K -> 2K 1%
- R202: footprint footprints:R_0402 -> footprints:R_0201_0603Metric; LCSC PN C105871 -> C138135
Connections:
- net +3V3: now also Y4.1, Y4.4 (VDD)
- net AUD_SD: now also U36.5, U36.6
- net AVCC3V3: now also U36.10 (V+)
- net GNDREF: now also U30.10 (NC_10), U30.3 (GND), U30.8 (GND), U36.4 (V-), Y4.2 (GND)
- net USBHOST_N: now also U30.2 (D1-)
- net USBHOST_P: now also U30.1 (D1+)
- net USBHOST_VBUS: now also U30.4 (D2+)
- net USB_VCC5V0: now also CR3.1
- net at C178.2, C179.1: now also U36.8 (-), U36.9
- net at C182.1, C183.1, Q10.1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: now also CR3.2
- net at C3.1, R12.2: now also U36.3 (+)
- net at C175.2, R16.2, R194.2: now also U36.1
- net at R16.1, R193.2: now also U36.2 (-)
- net at R201.1: now also Y4.3
- net at C177.1, R195.1: now also U36.7 (+)
Other:
- moved on the sheet: C184, C185, R201
