File: AUDIO.kicad_sch (KiCad schematic)
At the start: 47 parts, among them J15 USB-A-S-X-X-SM2, J9 SJ1-3525NG, Q10 DMG2305UX-13, U21 NC7WZ07P6X, U25 TPS2051BDBVR, U26 TUSB1210BRHBT, U30 TPD4E05U06DQAR, U36 AD8592ARM, Y4 ABM8G-26.000MHZ-18-D2Y-T

Commit message: post -production rework
Parts:
- removed C181: 1nF, footprints:C_0402, symbol Device:C
- added C52: GA342DR7GF102KW02L, footprints:CAPC4520X220N, symbol GA342DR7GF102KW02L:GA342DR7GF102KW02L
- R12: LCSC PN C852482 -> C270654
- R193, R200: now left out of the parts list
Connections:
- net GNDREF: now also C52.1
- net USB_SHIELD: now also C52.2
- net at R197.1: now also J9.3; no longer J9.2
- net at F2.2: now also J9.2; no longer J9.3
Other:
- moved on the sheet: R197
