File: ETHERNET.kicad_sch (KiCad schematic)
At the start: 73 parts, among them J12 HFJ11-1G01ERL, J13 503398-1892, U12 RTL8211F-CG, U13 TXS02612RTWR, U17 NC7WZ07P6X, U18 NL17SZ17XV5T2G, Y1 ABMM-25.000MHZ-B2-T

Commit message: update
Parts:
- C63, C79, C80: footprint footprints:C_0201_0603Metric -> footprints:C_0402
Connections:
- net VCC1V8_IO: now also R183.2; no longer R183.1
- net VCC1V8_IO_DLY: now also R183.1; no longer R183.2
Other:
- moved on the sheet: R179, R183
Changed lines of the file:
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@@
 		(color 0 0 0 0)
 	)
-	(bus_entry
-		(at 157.48 165.1)
-		(size 2.54 2.54)
-		(stroke
-			(width 0)
-			(type default)
-		)
-	)
 	(wire
 		(pts
@@
 	(symbol
 		(lib_id "Device:R_US")
-		(at 158.75 34.29 90)
-		(mirror x)
+		(at 158.75 34.29 270)
 		(unit 1)
 		(exclude_from_sim no)
@@
 		(dnp no)
 		(property "Reference" "R183"
-			(at 160.6173 36.4309 90)
+			(at 156.8827 36.4309 90)
 			(effects
 				(font
@@
 		)
 		(property "Value" "2.2K"
-			(at 159.3473 32.3669 90)
+			(at 158.1527 32.3669 90)
 			(effects
 				(font
@@
 		)
 		(property "Footprint" "footprints:R_0402"
-			(at 159.004 35.306 90)
+			(at 158.496 35.306 90)
 			(effects
 				(font
@@
 		(dnp no)
 		(property "Reference" "R166"
-			(at 29.972 49.53 90)
+			(at 27.432 50.038 90)
 			(effects
 				(font
@@
 		(lib_id "Device:C")
 		(at 106.68 143.51 0)
-		(mirror y)
 		(unit 1)
 		(exclude_from_sim no)
@@
 		(dnp no)
 		(property "Reference" "C80"
-			(at 103.378 142.748 0)
+			(at 109.982 142.748 0)
 			(effects
 				(font
@@
 		)
 		(property "Value" "100nF"
-			(at 104.394 145.288 0)
+			(at 108.966 145.288 0)
 			(effects
 				(font
@@
 			)
 		)
-		(property "Footprint" "footprints:C_0201_0603Metric"
-			(at 105.7148 147.32 0)
+		(property "Footprint" "footprints:C_0402"
+			(at 107.6452 147.32 0)
 			(effects
 				(font
@@
 	(symbol
 		(lib_id "Device:R_US")
-		(at 33.02 176.53 0)
-		(mirror x)
+		(at 33.02 176.53 180)
 		(unit 1)
 		(exclude_from_sim no)
@@
 		(dnp no)
 		(property "Reference" "R179"
-			(at 35.1609 174.6627 90)
+			(at 30.8791 174.6627 90)
 			(effects
 				(font
@@
 		)
 		(property "Value" "4.7K"
-			(at 31.0969 175.9327 90)
+			(at 34.9431 175.9327 90)
 			(effects
 				(font
@@
 		)
 		(property "Footprint" "footprints:R_0402"
-			(at 34.036 176.276 90)
+			(at 32.004 176.276 90)
 			(effects
 				(font
@@
 			)
 		)
-		(property "Footprint" "footprints:C_0201_0603Metric"
+		(property "Footprint" "footprints:C_0402"
 			(at 94.9452 147.32 0)
 			(effects
@@
 			)
 		)
-		(property "Footprint" "footprints:C_0201_0603Metric"
+		(property "Footprint" "footprints:C_0402"
 			(at 26.3652 151.13 0)
 			(effects
