File: ETHERNET.kicad_sch (KiCad schematic)
At the start: 73 parts, among them J12 HFJ11-1G01ERL, J13 503398-1892, U12 RTL8211F-CG, U13 TXS02612RTWR, U17 NC7WZ07P6X, U18 NL17SZ17XV5T2G, Y1 ABMM-25.000MHZ-B2-T

Commit message: new layout by abdul
Parts:
- C53, C54, C55, C56, C59, C65, C68, C70, C71, C73, C75, C78: footprint footprints:C_0402 -> footprints:C_0201_0603Metric
- R156, R157, R158, R159, R160, R161, R162, R163, R164, R165, R166, R167, R168, R169: footprint footprints:R_0402 -> footprints:R_0201_0603Metric
- R176, R177: value 390 -> 4.7k
Connections:
- net ETH_LD1: now also R175.2; no longer R174.2
- net ETH_LD2: now also R174.2; no longer R175.2
Other:
- moved on the sheet: L2
Changed lines of the file:
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@@
 	(wire
 		(pts
+			(xy 127 60.96) (xy 125.73 60.96)
+		)
+		(stroke
+			(width 0)
+			(type default)
+		)
+	)
+	(wire
+		(pts
 			(xy 57.15 50.8) (xy 52.07 50.8)
 		)
@@
 	(wire
 		(pts
-			(xy 146.05 60.96) (xy 147.32 60.96)
-		)
-		(stroke
-			(width 0)
-			(type default)
-		)
-	)
-	(wire
-		(pts
 			(xy 228.6 146.05) (xy 228.6 151.13)
 		)
@@
 		)
 	)
-	(global_label "ETH_LD1"
+	(global_label "ETH_LD2"
 		(shape bidirectional)
 		(at 147.32 114.3 0)
@@
 		)
 	)
-	(global_label "ETH_LD2"
+	(global_label "ETH_LD1"
 		(shape bidirectional)
 		(at 147.32 118.11 0)
@@
 			)
 		)
-		(property "Footprint" "footprints:C_0402"
+		(property "Footprint" "footprints:C_0201_0603Metric"
 			(at 157.1752 68.58 0)
 			(effects
@@
 			)
 		)
-		(property "Footprint" "footprints:C_0402"
+		(property "Footprint" "footprints:C_0201_0603Metric"
 			(at 229.5652 146.05 0)
 			(effects
@@
 		(fields_autoplaced yes)
 		(property "Reference" "U18"
-			(at 214.63 26.67 0)
+			(at 214.63 37.4649 0)
 			(effects
 				(font
 					(size 1.524 1.524)
 				)
+				(justify left)
 			)
 		)
 		(property "Value" "NL17SZ17XV5T2G"
-			(at 214.63 29.21 0)
+			(at 214.63 40.0049 0)
 			(effects
 				(font
 					(size 1.524 1.524)
 				)
+				(justify left)
 			)
 		)
@@
 			)
 		)
-		(property "Footprint" "footprints:C_0402"
+		(property "Footprint" "footprints:C_0201_0603Metric"
 			(at 240.9952 110.49 0)
 			(effects
@@
 			)
 		)
-		(property "Footprint" "footprints:C_0402"
+		(property "Footprint" "footprints:C_0201_0603Metric"
 			(at 240.9952 123.19 0)
 			(effects
@@
 			)
 		)
-		(property "Value" "390"
+		(property "Value" "4.7k"
 			(at 144.018 101.092 90)
 			(effects
@@
 			)
 		)
-		(property "Footprint" "footprints:R_0402"
+		(property "Footprint" "footprints:R_0201_0603Metric"
 			(at 30.226 53.086 90)
 			(effects
@@
 			)
 		)
-		(property "Footprint" "footprints:R_0402"
+		(property "Footprint" "footprints:R_0201_0603Metric"
 			(at 53.086 57.404 90)
 			(effects
@@
 			)
 		)
-		(property "Footprint" "footprints:R_0402"
+		(property "Footprint" "footprints:R_0201_0603Metric"
 			(at 48.006 56.134 90)
 			(effects
@@
 	)
 	(symbol
-		(lib_id "power:GNDREF")
-		(at 68.58 96.52 270)
-		(unit 1)
-		(exclude_from_sim no)
-		(in_bom yes)
-		(on_board yes)
-		(dnp no)
-		(fields_autoplaced yes)
-		(property "Reference" "#PWR0178"
-			(at 62.23 96.52 0)
-			(effects
-				(font
-					(size 1.27 1.27)
-				)
-				(hide yes)
-			)
-		)
-		(property "Value" "GNDREF"
-			(at 64.77 96.5199 90)
-			(effects
-				(font
-					(size 1.27 1.27)
-				)
-				(justify right)
-			)
-		)
-		(property "Footprint" ""
-			(at 68.58 96.52 0)
-			(effects
-				(font
-					(size 1.27 1.27)
-				)
-				(hide yes)
-			)
-		)
-		(property "Datasheet" ""
-			(at 68.58 96.52 0)
-			(effects
-				(font
-					(size 1.27 1.27)
-				)
-				(hide yes)
-			)
-		)
-		(property "Description" "Power symbol creates a global label with name \"GNDREF\" , reference supply ground"
-			(at 68.58 96.52 0)
-			(effects
-				(font
-					(size 1.27 1.27)
-				)
-				(hide yes)
-			)
-		)
-		(pin "1"
-		)
-		(instances
-			(project "FPGA-BOARDver3"
-				(path "/4a327bdf-04e5-4836-9c0a-5fb801c23f64/198f551b-0495-4dfe-9b6f-a7260738d114"
-					(reference "#PWR0178")
-					(unit 1)
-				)
-			)
-		)
-	)
-	(symbol
 		(lib_id "BLM18AG601SZ1D:BLM18AG601SZ1D")
 		(at 218.44 102.87 0)
@@
 			)
 		)
-		(property "Footprint" "footprints:R_0402"
+		(property "Footprint" "footprints:R_0201_0603Metric"
 			(at 30.226 75.946 90)
 			(effects
@@
 			)
 		)
-		(property "Footprint" "footprints:R_0402"
+		(property "Footprint" "footprints:R_0201_0603Metric"
 			(at 63.246 57.404 90)
 			(effects
@@
 		(lib_id "Device:C")
 		(at 232.41 106.68 0)
+		(mirror y)
 		(unit 1)
 		(exclude_from_sim no)
@@
 		(on_board yes)
 		(dnp no)
-		(fields_autoplaced yes)
 		(property "Reference" "C69"
-			(at 236.22 105.4099 0)
+			(at 228.6 105.4099 0)
 			(effects
 				(font
@@
 		)
 		(property "Value" "4.7uF"
-			(at 236.22 107.9499 0)
+			(at 228.6 107.9499 0)
 			(effects
 				(font
@@
 		)
 		(property "Footprint" "footprints:C_0402"
-			(at 233.3752 110.49 0)
+			(at 231.4448 110.49 0)
 			(effects
 				(font
@@
 			)
 		)
-		(property "Footprint" "footprints:R_0402"
+		(property "Footprint" "footprints:R_0201_0603Metric"
 			(at 54.356 84.074 90)
 			(effects
@@
 			)
 		)
-		(property "Footprint" "footprints:C_0402"
+		(property "Footprint" "footprints:C_0201_0603Metric"
 			(at 202.8952 123.19 0)
 			(effects
@@
 			)
 		)
-		(property "Footprint" "footprints:C_0402"
+		(property "Footprint" "footprints:C_0201_0603Metric"
 			(at 119.0752 29.21 0)
 			(effects
@@
 			)
 		)
-		(property "Footprint" "footprints:C_0402"
+		(property "Footprint" "footprints:C_0201_0603Metric"
 			(at 141.9352 29.21 0)
 			(effects
@@
 			)
 		)
-		(property "Footprint" "footprints:R_0402"
+		(property "Footprint" "footprints:R_0201_0603Metric"
 			(at 49.276 84.074 90)
 			(effects
@@
 			)
 		)
-		(property "Footprint" "footprints:R_0402"
+		(property "Footprint" "footprints:R_0201_0603Metric"
 			(at 30.226 70.866 90)
 			(effects
@@
 			)
 		)
-		(property "Footprint" "footprints:C_0402"
+		(property "Footprint" "footprints:C_0201_0603Metric"
 			(at 83.5152 26.67 0)
 			(effects
@@
 			)
 		)
-		(property "Footprint" "footprints:C_0402"
+		(property "Footprint" "footprints:C_0201_0603Metric"
 			(at 130.5052 29.21 0)
 			(effects
@@
 			)
 		)
-		(property "Footprint" "footprints:R_0402"
+		(property "Footprint" "footprints:R_0201_0603Metric"
 			(at 30.226 58.166 90)
 			(effects
@@
 			)
 		)
-		(property "Footprint" "footprints:C_0402"
+		(property "Footprint" "footprints:C_0201_0603Metric"
 			(at 248.6152 110.49 0)
 			(effects
@@
 			)
 		)
-		(property "Footprint" "footprints:R_0402"
+		(property "Footprint" "footprints:R_0201_0603Metric"
 			(at 68.326 20.066 90)
 			(effects
@@
 			)
 		)
-		(property "Footprint" "footprints:C_0402"
+		(property "Footprint" "footprints:C_0201_0603Metric"
 			(at 202.8952 110.49 0)
 			(effects
@@
 			)
 		)
-		(property "Footprint" "footprints:R_0402"
+		(property "Footprint" "footprints:R_0201_0603Metric"
 			(at 44.196 84.074 90)
 			(effects
@@
 	)
 	(symbol
+		(lib_name "NL17SZ17XV5T2G_Modified_1")
 		(lib_id "NL17SZ17XV5T2G:NL17SZ17XV5T2G_Modified")
 		(at 243.84 137.16 0)
@@
 			)
 		)
-		(property "Footprint" "footprints:R_0402"
+		(property "Footprint" "footprints:R_0201_0603Metric"
 			(at 30.226 82.296 90)
 			(effects
@@
 		(lib_id "Device:C")
 		(at 191.77 119.38 0)
+		(mirror y)
 		(unit 1)
 		(exclude_from_sim no)
@@
 		(on_board yes)
 		(dnp no)
-		(fields_autoplaced yes)
 		(property "Reference" "C72"
-			(at 195.58 118.1099 0)
+			(at 187.96 118.1099 0)
 			(effects
 				(font
@@
 		)
 		(property "Value" "4.7uF"
-			(at 195.58 120.6499 0)
+			(at 187.96 120.6499 0)
 			(effects
 				(font
@@
 		)
 		(property "Footprint" "footprints:C_0402"
-			(at 192.7352 123.19 0)
+			(at 190.8048 123.19 0)
 			(effects
 				(font
@@
 			)
 		)
-		(property "Footprint" "footprints:R_0402"
+		(property "Footprint" "footprints:R_0201_0603Metric"
 			(at 58.166 57.404 90)
 			(effects
@@
 			)
 		)
-		(property "Value" "390"
+		(property "Value" "4.7k"
 			(at 139.192 108.712 90)
 			(effects
@@
 			)
 		)
-		(property "Footprint" "footprints:R_0402"
+		(property "Footprint" "footprints:R_0201_0603Metric"
 			(at 30.226 63.246 90)
 			(effects
@@
 			)
 		)
-		(property "Footprint" "footprints:C_0402"
+		(property "Footprint" "footprints:C_0201_0603Metric"
 			(at 39.0652 92.71 0)
 			(effects
@@
 	(symbol
 		(lib_id "SRN4018-3R3M:SRN4018-3R3M")
-		(at 125.73 60.96 0)
+		(at 127 60.96 0)
 		(unit 1)
 		(exclude_from_sim no)
@@
 		(fields_autoplaced yes)
 		(property "Reference" "L2"
-			(at 135.89 54.61 0)
+			(at 137.16 54.61 0)
 			(effects
 				(font
@@
 		)
 		(property "Value" "SRN4018-3R3M"
-			(at 135.89 57.15 0)
+			(at 137.16 57.15 0)
 			(effects
 				(font
@@
 		)
 		(property "Footprint" "footprints:SRN4018"
-			(at 142.24 157.15 0)
+			(at 143.51 157.15 0)
 			(effects
 				(font
@@
 		)
 		(property "Datasheet" "https://www.bourns.com/docs/product-datasheets/srn4018.pdf?sfvrsn=528a0331_17"
-			(at 142.24 257.15 0)
+			(at 143.51 257.15 0)
 			(effects
 				(font
@@
 		)
 		(property "Description" "Inductor SMD 4x4 semi-shielded 3,3uH Bourns SRN4018 Series Shielded Wire-wound SMD Inductor with a Ferrite Core, 3.3 uH +/-20% Wire-Wound 2.2A rms Idc"
-			(at 125.73 60.96 0)
+			(at 127 60.96 0)
 			(effects
 				(font
@@
 		)
 		(property "Height" ""
-			(at 142.24 457.15 0)
+			(at 143.51 457.15 0)
 			(effects
 				(font
@@
 		)
 		(property "Mouser Part Number" "652-SRN4018-3R3M"
-			(at 142.24 557.15 0)
+			(at 143.51 557.15 0)
 			(effects
 				(font
@@
 		)
 		(property "Mouser Price/Stock" "https://www.mouser.co.uk/ProductDetail/Bourns/SRN4018-3R3M?qs=UvjENeDOEecJUn4TJeWI1g%3D%3D"
-			(at 142.24 657.15 0)
+			(at 143.51 657.15 0)
 			(effects
 				(font
@@
 		)
 		(property "Manufacturer_Name" "Bourns"
-			(at 142.24 757.15 0)
+			(at 143.51 757.15 0)
 			(effects
 				(font
@@
 		)
 		(property "Manufacturer_Part_Number" "SRN4018-3R3M"
-			(at 142.24 857.15 0)
+			(at 143.51 857.15 0)
 			(effects
 				(font
@@
 		)
 		(property "LCSC PN" "C2044390"
-			(at 125.73 60.96 0)
+			(at 127 60.96 0)
 			(effects
 				(font

Commit message: weekend update
Parts:
- C62: footprint footprints:C_0402 -> footprints:C_0201_0603Metric
Changed lines of the file:
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@@
 			)
 		)
-		(property "Footprint" "footprints:C_0402"
+		(property "Footprint" "footprints:C_0201_0603Metric"
 			(at 61.9252 138.43 0)
 			(effects

Commit message: update
Parts:
- C63, C79, C80: footprint footprints:C_0402 -> footprints:C_0201_0603Metric
Connections:
- net VCC1V8_IO: now also R183.1; no longer R183.2
- net VCC1V8_IO_DLY: now also R183.2; no longer R183.1
Other:
- moved on the sheet: R179, R183
Changed lines of the file:
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@@
 		(color 0 0 0 0)
 	)
+	(bus_entry
+		(at 157.48 165.1)
+		(size 2.54 2.54)
+		(stroke
+			(width 0)
+			(type default)
+		)
+	)
 	(wire
 		(pts
@@
 	(symbol
 		(lib_id "Device:R_US")
-		(at 158.75 34.29 270)
+		(at 158.75 34.29 90)
+		(mirror x)
 		(unit 1)
 		(exclude_from_sim no)
@@
 		(dnp no)
 		(property "Reference" "R183"
-			(at 156.8827 36.4309 90)
+			(at 160.6173 36.4309 90)
 			(effects
 				(font
@@
 		)
 		(property "Value" "2.2K"
-			(at 158.1527 32.3669 90)
+			(at 159.3473 32.3669 90)
 			(effects
 				(font
@@
 		)
 		(property "Footprint" "footprints:R_0402"
-			(at 158.496 35.306 90)
+			(at 159.004 35.306 90)
 			(effects
 				(font
@@
 		(dnp no)
 		(property "Reference" "R166"
-			(at 27.432 50.038 90)
+			(at 29.972 49.53 90)
 			(effects
 				(font
@@
 		(lib_id "Device:C")
 		(at 106.68 143.51 0)
+		(mirror y)
 		(unit 1)
 		(exclude_from_sim no)
@@
 		(dnp no)
 		(property "Reference" "C80"
-			(at 109.982 142.748 0)
+			(at 103.378 142.748 0)
 			(effects
 				(font
@@
 		)
 		(property "Value" "100nF"
-			(at 108.966 145.288 0)
+			(at 104.394 145.288 0)
 			(effects
 				(font
@@
 			)
 		)
-		(property "Footprint" "footprints:C_0402"
-			(at 107.6452 147.32 0)
+		(property "Footprint" "footprints:C_0201_0603Metric"
+			(at 105.7148 147.32 0)
 			(effects
 				(font
@@
 	(symbol
 		(lib_id "Device:R_US")
-		(at 33.02 176.53 180)
+		(at 33.02 176.53 0)
+		(mirror x)
 		(unit 1)
 		(exclude_from_sim no)
@@
 		(dnp no)
 		(property "Reference" "R179"
-			(at 30.8791 174.6627 90)
+			(at 35.1609 174.6627 90)
 			(effects
 				(font
@@
 		)
 		(property "Value" "4.7K"
-			(at 34.9431 175.9327 90)
+			(at 31.0969 175.9327 90)
 			(effects
 				(font
@@
 		)
 		(property "Footprint" "footprints:R_0402"
-			(at 32.004 176.276 90)
+			(at 34.036 176.276 90)
 			(effects
 				(font
@@
 			)
 		)
-		(property "Footprint" "footprints:C_0402"
+		(property "Footprint" "footprints:C_0201_0603Metric"
 			(at 94.9452 147.32 0)
 			(effects
@@
 			)
 		)
-		(property "Footprint" "footprints:C_0402"
+		(property "Footprint" "footprints:C_0201_0603Metric"
 			(at 26.3652 151.13 0)
 			(effects

Commit message: ready for manufacturing
Parts:
- removed L2: SRN4018-3R3M, footprints:SRN4018, symbol SRN4018-3R3M:SRN4018-3R3M
- added L8: NR4018T3R3M, footprints:NR4018T3R3M, symbol NR4018T3R3M:NR4018T3R3M
- C53, C54, C55, C56, C63, C65, C68, C70, C71, C73, C75, C78, C79, C80: LCSC PN c1525 -> c307380
- C57, C76: footprint footprints:C_0402 -> footprints:C_0201_0603Metric; LCSC PN c1525 -> c307380
- C58, C64, C67, C69, C72, C74, C77: LCSC PN c23733 -> C2858031
- C59, C62: LCSC PN c472451 -> C161381
- C60, C61: footprint footprints:C_0402 -> footprints:C_0201_0603Metric; LCSC PN c472451 -> C161381
- C66: LCSC PN c14442 -> C77018
- FL3, FL4: value 600Ohm/100MHz -> 600Ohm/100Mhz
- R156: footprint footprints:R_0201_0603Metric -> footprints:R_0402
- R157, R158, R159: LCSC PN C138040 -> C327393
- R160, R167, R168, R169: LCSC PN C105871 -> C138135
- R161, R162, R163, R164, R165, R166: LCSC PN C106231 -> c106228
- R176, R177: LCSC PN C137997 -> C105871
- R178, R179, R186: footprint footprints:R_0402 -> footprints:R_0201_0603Metric; LCSC PN C105871 -> C138135
Connections:
- net ETH_VCC1V0: now also L8.2
- net at R180.1, U12.30 (REG_OUT/LDO_OUT): now also L8.1
