File: ETHERNET.kicad_sch (KiCad schematic)
At the start: 73 parts, among them J12 HFJ11-1G01ERL, J13 503398-1892, U12 RTL8211F-CG, U13 TXS02612RTWR, U17 NC7WZ07P6X, U18 NL17SZ17XV5T2G, Y1 ABMM-25.000MHZ-B2-T

Commit message: post -production rework
Parts:
- removed C66: 1nF, footprints:C_0402, symbol Device:C
- removed U17: NC7WZ07P6X, footprints:NC7WZ07P6X, symbol NC7WZ07P6X:NC7WZ07P6X_modified
- added C222: GA342DR7GF102KW02L, footprints:CAPC4520X220N, symbol GA342DR7GF102KW02L:GA342DR7GF102KW02L
- added U20: NC7WZ07P6X, footprints:NC7WZ07P6X, symbol NC7WZ07P6X:NC7WZ07P6X_modified
- C59, C62, R168, R180, R186: now left out of the parts list
- D28, D32, D33: LCSC PN C434449 -> C130723
Connections:
- net +1V8: now also U20.5 (VCC)
- net ETH_RST_B: now also U20.6
- net ETH_TD1_N: now also J12.6; no longer J12.4
- net ETH_TD2_N: now also J12.5; no longer J12.6
- net ETH_TD2_P: now also J12.4; no longer J12.5
- net GNDREF: now also C222.1, U20.2 (GND), U20.3
- net SHIELD: now also C222.2
- net VCC1V8_IO_EDGE: now also U20.1
Other:
- moved on the sheet: R182
