File: POWER_REGULATION.kicad_sch (KiCad schematic)
At the start: 43 parts, among them J1 PJ-102AH, J17 Conn_01x02_Pin, J2 Conn_01x01_Pin, J3 Conn_01x03_Pin, Q7 DMG2305UX-13, U14 TLV62130RGTT, U16 REF3012

Commit message: update
Parts:
- C18, C32: footprint footprints:C_0201_0603Metric -> footprints:C_0402
Changed lines of the file:
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@@
 			)
 		)
-		(property "Footprint" "footprints:C_0201_0603Metric"
+		(property "Footprint" "footprints:C_0402"
 			(at 55.5752 129.54 0)
 			(effects
@@
 			)
 		)
-		(property "Footprint" "footprints:C_0201_0603Metric"
+		(property "Footprint" "footprints:C_0402"
 			(at 84.7852 135.89 0)
 			(effects
