File: POWER_REGULATION.kicad_sch (KiCad schematic)
At the start: 41 parts, among them J1 PJ-102AH, J17 Conn_01x02_Pin, J2 Conn_01x01_Pin, J3 Conn_01x03_Pin, Q7 DMG2305UX-13, U14 TLV62130RGTT, U15 LP5907MFX-3.3, U16 REF3012

Commit message: new layout by abdul
Parts:
- removed L3: NR5040T4R7N / 4.7uH, footprints:IND_TAIYO_NR5040_TAY, symbol NR5040T4R7N:NR5040T4R7N
- removed U15: LP5907MFX-3.3, footprints:SOT-23-5, symbol Regulator_Linear:LP5907MFX-3.3
- added C234: 100nF, footprints:C_0201_0603Metric, symbol Device:C
- added C7: 4.7uF, footprints:C_0402, symbol Device:C
- added FL9: 600Ohm/100MHz, footprints:BEADC1608X95N, symbol BLM18AG601SZ1D:BLM18AG601SZ1D
- added L4: NR5040T2R2N/2.2uH, footprints:IND_TAIYO_NR5040_TAY, symbol 2025-03-04_21-33-04:NR5040T2R2N
- C19: value 1uF -> 100nF; footprint footprints:C_0402 -> footprints:C_0201_0603Metric; LCSC PN c14445 -> c1525
- C192, C193, C194, C195, C196, C197, C198, C29, C31: footprint footprints:C_0402 -> footprints:C_0805
- C199: value 10uF -> 100nF; footprint footprints:C_0402 -> footprints:C_0201_0603Metric; LCSC PN c315248 -> c1525
- C20: value 1uF -> 4.7uF; LCSC PN c14445 -> c23733
- C26: footprint footprints:C_0402 -> footprints:C_0201_0603Metric; LCSC PN c92361 -> C88915
- C28: footprint footprints:C_0402 -> footprints:C_0201_0603Metric
Connections:
- net +5V: no longer C19.1
- net AVCC3V3: now also C199.1, C234.1, FL9.2
- net GNDREF: now also C234.2, C7.2
- net REG5V0: now also L4.1
- net VU: no longer C199.1
- net at U14.1 (SW@1), U14.2 (SW@2), U14.3 (SW@3): now also L4.2
- new net +3V3: C19.1, C7.1, FL9.1

Commit message: update
Parts:
- C18, C32: footprint footprints:C_0402 -> footprints:C_0201_0603Metric
Changed lines of the file:
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@@
 			)
 		)
-		(property "Footprint" "footprints:C_0402"
+		(property "Footprint" "footprints:C_0201_0603Metric"
 			(at 55.5752 129.54 0)
 			(effects
@@
 			)
 		)
-		(property "Footprint" "footprints:C_0402"
+		(property "Footprint" "footprints:C_0201_0603Metric"
 			(at 84.7852 135.89 0)
 			(effects

Commit message: ready for manufacturing
Parts:
- removed CR4: DDZ9699-7, footprints:ZDO_SOD123_DIO, symbol DDZ9699-7:DDZ9699-7
- added CR7: BZT52C12-7-F, footprints:SOD123_DIO, symbol BZT52C12_7_F:BZT52C12-7-F
- added J18: +3V3, footprints:PinHeader_1x01_P2.54mm_Vertical, symbol Connector:Conn_01x01_Pin
- added J19: +1V8, footprints:PinHeader_1x01_P2.54mm_Vertical, symbol Connector:Conn_01x01_Pin
- added J20: +1V5, footprints:PinHeader_1x01_P2.54mm_Vertical, symbol Connector:Conn_01x01_Pin
- added J21: +1V0, footprints:PinHeader_1x01_P2.54mm_Vertical, symbol Connector:Conn_01x01_Pin
- added J22: VCC_1V8IO, footprints:PinHeader_1x01_P2.54mm_Vertical, symbol Connector:Conn_01x01_Pin
- C18, C19, C199, C234, C28, C32: LCSC PN c1525 -> c307380
- C192, C193, C194, C195, C196, C197, C198: value 10uF -> 10uF 10V; LCSC PN c315248 -> C15850
- C20, C7: LCSC PN c23733 -> C2858031
- C21: value 1uF -> 1uF 10V; LCSC PN c14445 -> C52923
- C26: LCSC PN C88915 -> C5383023
- C27: value 4.7uF/10V -> 4.7uF; LCSC PN c23733 -> C2858031
- C29: footprint footprints:C_0805 -> footprints:C_0402
- C30: value 0.1uF -> 100nF 10V; LCSC PN c1525 -> C77020
- C31: value 10uF/10V -> 10uF 10V; LCSC PN c315248 -> C15850
- FL2, FL5: LCSC PN digi/mouser -> C19330
- FL9: value 600Ohm/100MHz -> 600Ohm/100Mhz
- J1: LCSC PN C3096093 -> (none)
- J17, J3: LCSC PN digi/mouser -> (none)
- J2: value Conn_01x01_Pin -> GND; LCSC PN digi/mouser -> (none)
- L4: LCSC PN (none) -> C223063
- R83: value 100k -> 100K
- R85: value 20k -> 20K 1%
- R86: value 10K -> 10K 1%
- R89: value 10k/1% -> 10K 1%
Connections:
- net +1V8: now also J19.1 (Pin_1)
- net +3V3: now also J18.1 (Pin_1)
- net VBUS: now also CR7.1
- net at C27.2, Q7.1, R83.2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: now also CR7.2
- new net +1V0: J21.1 (Pin_1)
- new net +1V5: J20.1 (Pin_1)
- new net VCC1V8_IO: J22.1 (Pin_1)
