File: POWER_REGULATION.kicad_sch (KiCad schematic)
At the start: 48 parts, among them J1 PJ-102AH, J17 Conn_01x02_Pin, J18 +3V3, J19 +1V8, J2 GND, J20 +1V5, J21 +1V0, J22 VCC_1V8IO, J3 Conn_01x03_Pin, Q7 DMG2305UX-13, U14 TLV62130RGTT, U16 REF3012

Commit message: post -production rework
Parts:
- removed J19: +1V8, footprints:PinHeader_1x01_P2.54mm_Vertical, symbol Connector:Conn_01x01_Pin
- R88: LCSC PN C852893 -> C5126210
- R91: now left out of the parts list
Other:
- moved on the sheet: J21, J22
