File: POWER_REGULATION2.kicad_sch (KiCad schematic)
At the start: 72 parts, among them Q8 FDV301N, U19 NL17SZ17XV5T2G, U20 FPF1018, U21 NC7WZ07P6X, U22 TPS65400RGZT, U9 SIP32510DT-T1-GE3

Commit message: new layout by abdul
Parts:
- C139, C140, C141, C142: value 22uF -> 22uF/10V; footprint footprints:C_0402 -> footprints:C_0805
- C147, C148, C149, C150, C151, C152, C153, C154, C157, C158, C159, C160, C161, C163, C166, C169, C33: footprint footprints:C_0402 -> footprints:C_0201_0603Metric
- C156, C164, C167, C170, C200: footprint footprints:C_0402 -> footprints:C_0805
- L5: value SRP6540-1R5M -> SRP6540-1R5M 1.5uH
- R94: footprint footprints:R_0402 -> footprints:R_0201_0603Metric
Connections:
- net at U22.38 (I2CADDR): now also R206.2
- net at U22.41 (I2CALERT): no longer R206.2
Changed lines of the file:
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@@
 	)
 	(junction
+		(at 21.59 170.18)
+		(diameter 0)
+		(color 0 0 0 0)
+	)
+	(junction
 		(at 120.65 52.07)
 		(diameter 0)
@@
 	(wire
 		(pts
-			(xy 20.32 170.18) (xy 24.13 170.18)
+			(xy 20.32 170.18) (xy 21.59 170.18)
 		)
 		(stroke
@@
 	(wire
 		(pts
+			(xy 21.59 176.53) (xy 21.59 170.18)
+		)
+		(stroke
+			(width 0)
+			(type default)
+		)
+	)
+	(wire
+		(pts
 			(xy 83.82 39.37) (xy 90.17 39.37)
 		)
@@
 	(wire
 		(pts
+			(xy 21.59 170.18) (xy 24.13 170.18)
+		)
+		(stroke
+			(width 0)
+			(type default)
+		)
+	)
+	(wire
+		(pts
 			(xy 133.35 46.99) (xy 140.97 46.99)
 		)
@@
 	(wire
 		(pts
+			(xy 24.13 176.53) (xy 21.59 176.53)
+		)
+		(stroke
+			(width 0)
+			(type default)
+		)
+	)
+	(wire
+		(pts
 			(xy 186.69 118.11) (xy 218.44 118.11)
 		)
@@
 	(wire
 		(pts
-			(xy 24.13 170.18) (xy 24.13 176.53)
-		)
-		(stroke
-			(width 0)
-			(type default)
-		)
-	)
-	(wire
-		(pts
 			(xy 90.17 105.41) (xy 90.17 100.33)
 		)
@@
 			)
 		)
-		(property "Footprint" "footprints:C_0402"
+		(property "Footprint" "footprints:C_0805"
 			(at 240.9952 77.47 0)
 			(effects
@@
 			)
 		)
-		(property "Footprint" "footprints:C_0402"
+		(property "Footprint" "footprints:C_0201_0603Metric"
 			(at 100.33 38.4048 0)
 			(effects
@@
 			)
 		)
-		(property "Footprint" "footprints:C_0402"
+		(property "Footprint" "footprints:C_0201_0603Metric"
 			(at 133.35 46.0248 0)
 			(effects
@@
 			)
 		)
-		(property "Value" "22uF"
+		(property "Value" "22uF/10V"
 			(at 220.98 20.3199 0)
 			(effects
@@
 			)
 		)
-		(property "Footprint" "footprints:C_0402"
+		(property "Footprint" "footprints:C_0805"
 			(at 218.1352 22.86 0)
 			(effects
@@
 			)
 		)
-		(property "Footprint" "footprints:C_0402"
+		(property "Footprint" "footprints:C_0201_0603Metric"
 			(at 133.35 58.7248 0)
 			(effects
@@
 			)
 		)
-		(property "Footprint" "footprints:C_0402"
+		(property "Footprint" "footprints:C_0805"
 			(at 240.9952 50.8 0)
 			(effects
@@
 			)
 		)
-		(property "Value" "SRP6540-1R5M"
+		(property "Value" "SRP6540-1R5M 1.5uH"
 			(at 209.55 59.69 0)
 			(effects
@@
 		(on_board yes)
 		(dnp no)
-		(fields_autoplaced yes)
 		(property "Reference" "C139"
-			(at 194.31 17.7799 0)
+			(at 184.658 17.018 0)
 			(effects
 				(font
@@
 			)
 		)
-		(property "Value" "22uF"
-			(at 194.31 20.3199 0)
+		(property "Value" "22uF/10V"
+			(at 179.832 19.558 0)
 			(effects
 				(font
@@
 			)
 		)
-		(property "Footprint" "footprints:C_0402"
+		(property "Footprint" "footprints:C_0805"
 			(at 191.4652 22.86 0)
 			(effects
@@
 			)
 		)
-		(property "Footprint" "footprints:C_0402"
+		(property "Footprint" "footprints:C_0201_0603Metric"
 			(at 107.95 104.4448 0)
 			(effects
@@
 		(on_board yes)
 		(dnp no)
-		(fields_autoplaced yes)
 		(property "Reference" "S1"
 			(at 152.4 173.9899 0)
@@
 			)
 		)
-		(property "Footprint" "footprints:C_0402"
+		(property "Footprint" "footprints:C_0805"
 			(at 240.9952 123.19 0)
 			(effects
@@
 			)
 		)
-		(property "Footprint" "footprints:R_0402"
+		(property "Footprint" "footprints:R_0201_0603Metric"
 			(at 115.316 167.894 90)
 			(effects
@@
 			)
 		)
-		(property "Footprint" "footprints:C_0402"
+		(property "Footprint" "footprints:C_0805"
 			(at 249.8852 77.47 0)
 			(effects
@@
 			)
 		)
-		(property "Footprint" "footprints:C_0402"
+		(property "Footprint" "footprints:C_0201_0603Metric"
 			(at 100.33 84.1248 0)
 			(effects
@@
 			)
 		)
-		(property "Footprint" "footprints:C_0402"
+		(property "Footprint" "footprints:C_0201_0603Metric"
 			(at 133.35 106.9848 0)
 			(effects
@@
 			)
 		)
-		(property "Footprint" "footprints:C_0402"
+		(property "Footprint" "footprints:C_0201_0603Metric"
 			(at 229.5652 118.11 0)
 			(effects
@@
 			)
 		)
-		(property "Footprint" "footprints:C_0402"
+		(property "Footprint" "footprints:C_0201_0603Metric"
 			(at 41.6052 38.1 0)
 			(effects
@@
 			)
 		)
-		(property "Footprint" "footprints:C_0402"
+		(property "Footprint" "footprints:C_0201_0603Metric"
 			(at 100.33 99.3648 0)
 			(effects
@@
 			)
 		)
-		(property "Footprint" "footprints:C_0402"
+		(property "Footprint" "footprints:C_0201_0603Metric"
 			(at 132.08 91.7448 0)
 			(effects
@@
 		(on_board yes)
 		(dnp no)
-		(fields_autoplaced yes)
 		(property "Reference" "C140"
-			(at 203.2 17.7799 0)
+			(at 194.818 17.018 0)
 			(effects
 				(font
@@
 			)
 		)
-		(property "Value" "22uF"
-			(at 203.2 20.3199 0)
+		(property "Value" "22uF/10V"
+			(at 193.294 20.574 0)
 			(effects
 				(font
@@
 			)
 		)
-		(property "Footprint" "footprints:C_0402"
+		(property "Footprint" "footprints:C_0805"
 			(at 200.3552 22.86 0)
 			(effects
@@
 			)
 		)
-		(property "Footprint" "footprints:C_0402"
+		(property "Footprint" "footprints:C_0201_0603Metric"
 			(at 229.5652 45.72 0)
 			(effects
@@
 		(on_board yes)
 		(dnp no)
-		(fields_autoplaced yes)
 		(property "Reference" "C141"
-			(at 212.09 17.7799 0)
+			(at 203.708 17.018 0)
 			(effects
 				(font
@@
 			)
 		)
-		(property "Value" "22uF"
-			(at 212.09 20.3199 0)
+		(property "Value" "22uF/10V"
+			(at 203.708 20.066 0)
 			(effects
 				(font
@@
 			)
 		)
-		(property "Footprint" "footprints:C_0402"
+		(property "Footprint" "footprints:C_0805"
 			(at 209.2452 22.86 0)
 			(effects
@@
 			)
 		)
-		(property "Footprint" "footprints:C_0402"
+		(property "Footprint" "footprints:C_0201_0603Metric"
 			(at 107.95 89.2048 0)
 			(effects
@@
 			)
 		)
-		(property "Footprint" "footprints:C_0402"
+		(property "Footprint" "footprints:C_0201_0603Metric"
 			(at 107.95 43.4848 0)
 			(effects
@@
 		(dnp no)
 		(property "Reference" "C165"
-			(at 195.58 59.6899 0)
+			(at 192.024 55.626 0)
 			(effects
 				(font
@@
 		)
 		(property "Value" "100nF"
-			(at 195.58 62.2299 0)
+			(at 193.04 56.896 0)
 			(effects
 				(font
@@
 			)
 		)
-		(property "Footprint" "footprints:C_0402"
+		(property "Footprint" "footprints:C_0201_0603Metric"
 			(at 229.5652 72.39 0)
 			(effects
@@
 			)
 		)
-		(property "Footprint" "footprints:C_0402"
+		(property "Footprint" "footprints:C_0201_0603Metric"
 			(at 229.5652 95.25 0)
 			(effects
@@
 			)
 		)
-		(property "Footprint" "footprints:C_0402"
+		(property "Footprint" "footprints:C_0805"
 			(at 240.9952 100.33 0)
 			(effects
@@
 			)
 		)
-		(property "Footprint" "footprints:C_0402"
+		(property "Footprint" "footprints:C_0201_0603Metric"
 			(at 100.33 51.1048 0)
 			(effects
@@
 			)
 		)
-		(property "Footprint" "footprints:C_0402"
+		(property "Footprint" "footprints:C_0201_0603Metric"
 			(at 107.95 56.1848 0)
 			(effects

Commit message: update
Parts:
- C155, C162, C165, C168: footprint footprints:C_0402 -> footprints:C_0201_0603Metric
Changed lines of the file:
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@@
 			)
 		)
-		(property "Footprint" "footprints:C_0402"
+		(property "Footprint" "footprints:C_0201_0603Metric"
 			(at 192.7352 110.49 0)
 			(effects
@@
 			)
 		)
-		(property "Footprint" "footprints:C_0402"
+		(property "Footprint" "footprints:C_0201_0603Metric"
 			(at 192.7352 62.23 0)
 			(effects
@@
 			)
 		)
-		(property "Footprint" "footprints:C_0402"
+		(property "Footprint" "footprints:C_0201_0603Metric"
 			(at 192.7352 87.63 0)
 			(effects
@@
 		(lib_id "Device:C")
 		(at 228.6 91.44 0)
+		(mirror y)
 		(unit 1)
 		(exclude_from_sim no)
@@
 		(on_board yes)
 		(dnp no)
-		(fields_autoplaced yes)
 		(property "Reference" "C163"
-			(at 232.41 90.1699 0)
+			(at 224.79 90.1699 0)
 			(effects
 				(font
@@
 		)
 		(property "Value" "10pF"
-			(at 232.41 92.7099 0)
+			(at 224.79 92.7099 0)
 			(effects
 				(font
@@
 		)
 		(property "Footprint" "footprints:C_0201_0603Metric"
-			(at 229.5652 95.25 0)
+			(at 227.6348 95.25 0)
 			(effects
 				(font
@@
 			)
 		)
-		(property "Footprint" "footprints:C_0402"
+		(property "Footprint" "footprints:C_0201_0603Metric"
 			(at 192.7352 35.56 0)
 			(effects

Commit message: update
Parts:
- C155, C162, C165, C168: footprint footprints:C_0201_0603Metric -> footprints:C_0402
Changed lines of the file:
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@@
 			)
 		)
-		(property "Footprint" "footprints:C_0201_0603Metric"
+		(property "Footprint" "footprints:C_0402"
 			(at 192.7352 110.49 0)
 			(effects
@@
 			)
 		)
-		(property "Footprint" "footprints:C_0201_0603Metric"
+		(property "Footprint" "footprints:C_0402"
 			(at 192.7352 62.23 0)
 			(effects
@@
 			)
 		)
-		(property "Footprint" "footprints:C_0201_0603Metric"
+		(property "Footprint" "footprints:C_0402"
 			(at 192.7352 87.63 0)
 			(effects
@@
 		(lib_id "Device:C")
 		(at 228.6 91.44 0)
-		(mirror y)
 		(unit 1)
 		(exclude_from_sim no)
@@
 		(on_board yes)
 		(dnp no)
+		(fields_autoplaced yes)
 		(property "Reference" "C163"
-			(at 224.79 90.1699 0)
+			(at 232.41 90.1699 0)
 			(effects
 				(font
@@
 		)
 		(property "Value" "10pF"
-			(at 224.79 92.7099 0)
+			(at 232.41 92.7099 0)
 			(effects
 				(font
@@
 		)
 		(property "Footprint" "footprints:C_0201_0603Metric"
-			(at 227.6348 95.25 0)
+			(at 229.5652 95.25 0)
 			(effects
 				(font
@@
 			)
 		)
-		(property "Footprint" "footprints:C_0201_0603Metric"
+		(property "Footprint" "footprints:C_0402"
 			(at 192.7352 35.56 0)
 			(effects
