File: POWER_REGULATION2.kicad_sch (KiCad schematic)
At the start: 72 parts, among them Q8 FDV301N, U19 NL17SZ17XV5T2G, U20 FPF1018, U21 NC7WZ07P6X, U22 TPS65400RGZT, U9 SIP32510DT-T1-GE3

Commit message: ready for manufacturing
Parts:
- removed L10: TYS60282R2N-10/2.2uH, footprints:IND_TYS60282_LRD, symbol 2025-03-18_07-11-26:TYS60282R2N-10
- removed U20: FPF1018, footprints:MLP6_2X2_ONS, symbol FPF1018:FPF1018
- added C203: 1uF 10V, footprints:C_0402, symbol Device:C
- added L3: NR5040T2R2N/2.2uH, footprints:IND_TAIYO_NR5040_TAY, symbol 2025-03-04_21-33-04:NR5040T2R2N
- added U40: TPS22918DBVR, footprints:DBV6_TEX, symbol TPS22918DBVR:TPS22918DBVR
- C139, C140, C141, C142: LCSC PN c415703 -> C602037
- C143: value 10uF/10V -> 10uF 10V; footprint footprints:C_0402 -> footprints:C_0805; LCSC PN c315248 -> C15850
- C144: value 1uF/10V -> 1uF 10V; LCSC PN c14445 -> C52923
- C145: footprint footprints:C_0402 -> footprints:C_0603; LCSC PN c51412 -> C528975
- C146: value 4.7uF/10V -> 4.7uF; LCSC PN c23733 -> C2858031
- C147: LCSC PN c23967 -> C2184288
- C148, C154, C157, C160: LCSC PN c472437 -> C161475
- C149, C151, C153, C159, C161, C163, C166, C169: LCSC PN c307440 -> C76921
- C150: LCSC PN c1527 -> C3843470
- C152: LCSC PN c393671 -> C18213195
- C155, C162, C165, C168, C33: LCSC PN c1525 -> c307380
- C156, C164, C167, C170, C200: value 22uF -> 22uF/10V; LCSC PN c415703 -> C602037
- C158: LCSC PN c13533 -> C2184280
- C171, C174: footprint footprints:C_0402 -> footprints:C_0201_0603Metric; LCSC PN c1525 -> c307380
- C172, C81: LCSC PN c23733 -> C2858031
- C173: value 1uF -> 1uF 10V; LCSC PN c14445 -> C52923
- D25: LCSC PN C434449 -> C21260817
- L6, L7: LCSC PN C223063 -> C223064
- R105: value 20K/1% -> 20K 1%
- R206, R99: value 10K -> 10K 1%
- R94: LCSC PN C137948 -> C307010
- U9: LCSC PN C145264 -> (none)
Connections:
- net +1V0: now also L3.1
- net +1V8: now also U40.1 (VIN)
- net GNDREF: now also C203.2, U40.2 (GND), U40.4 (CT), U40.5 (QOD)
- net PG_ALL: now also U40.3 (ON)
- net VCC1V8_IO: now also C203.1, U40.6 (VOUT)
- net at C168.2, U22.2 (SW1), U22.3 (SW1__1)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: now also L3.2
