File: DDR3.kicad_sch (KiCad schematic)
At the start: 24 parts, among them IC1 IS43TR16256B-125KBLI

Commit message: new layout by abdul
Parts:
- C36, C37, C38, C39, C40, C41, C42, C43, C44, C45, C46, C47, C48, C49, C50, C51: footprint footprints:C_0402 -> footprints:C_0201_0603Metric
- C82, C83: footprint footprints:C_0402 -> footprints:C_0201_0603Metric; LCSC PN c92361 -> C88915
- C84: value 4.7nF -> 4.7uF
Changed lines of the file:
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@@
 			)
 		)
-		(property "Footprint" "footprints:C_0402"
+		(property "Footprint" "footprints:C_0201_0603Metric"
 			(at 204.1652 66.04 0)
 			(effects
@@
 			)
 		)
-		(property "Footprint" "footprints:C_0402"
+		(property "Footprint" "footprints:C_0201_0603Metric"
 			(at 234.6452 85.09 0)
 			(effects
@@
 			)
 		)
-		(property "Footprint" "footprints:C_0402"
+		(property "Footprint" "footprints:C_0201_0603Metric"
 			(at 183.8452 66.04 0)
 			(effects
@@
 			)
 		)
-		(property "Footprint" "footprints:C_0402"
+		(property "Footprint" "footprints:C_0201_0603Metric"
 			(at 244.8052 85.09 0)
 			(effects
@@
 			)
 		)
-		(property "Footprint" "footprints:C_0402"
+		(property "Footprint" "footprints:C_0201_0603Metric"
 			(at 183.8452 104.14 0)
 			(effects
@@
 			)
 		)
-		(property "LCSC PN" "c92361"
+		(property "LCSC PN" "C88915"
 			(at 182.88 100.33 0)
 			(effects
@@
 			)
 		)
-		(property "Footprint" "footprints:C_0402"
+		(property "Footprint" "footprints:C_0201_0603Metric"
 			(at 254.9652 85.09 0)
 			(effects
@@
 			)
 		)
-		(property "Footprint" "footprints:C_0402"
+		(property "Footprint" "footprints:C_0201_0603Metric"
 			(at 214.3252 85.09 0)
 			(effects
@@
 			)
 		)
-		(property "Footprint" "footprints:C_0402"
+		(property "Footprint" "footprints:C_0201_0603Metric"
 			(at 214.3252 66.04 0)
 			(effects
@@
 			)
 		)
-		(property "Footprint" "footprints:C_0402"
+		(property "Footprint" "footprints:C_0201_0603Metric"
 			(at 194.0052 66.04 0)
 			(effects
@@
 			)
 		)
-		(property "Footprint" "footprints:C_0402"
+		(property "Footprint" "footprints:C_0201_0603Metric"
 			(at 183.8452 85.09 0)
 			(effects
@@
 			)
 		)
-		(property "Footprint" "footprints:C_0402"
+		(property "Footprint" "footprints:C_0201_0603Metric"
 			(at 224.4852 85.09 0)
 			(effects
@@
 			)
 		)
-		(property "Footprint" "footprints:C_0402"
+		(property "Footprint" "footprints:C_0201_0603Metric"
 			(at 194.0052 85.09 0)
 			(effects
@@
 			)
 		)
-		(property "Footprint" "footprints:C_0402"
+		(property "Footprint" "footprints:C_0201_0603Metric"
 			(at 254.9652 66.04 0)
 			(effects
@@
 			)
 		)
-		(property "Footprint" "footprints:C_0402"
+		(property "Footprint" "footprints:C_0201_0603Metric"
 			(at 194.0052 104.14 0)
 			(effects
@@
 			)
 		)
-		(property "LCSC PN" "c92361"
+		(property "LCSC PN" "C88915"
 			(at 193.04 100.33 0)
 			(effects
@@
 			)
 		)
-		(property "Footprint" "footprints:C_0402"
+		(property "Footprint" "footprints:C_0201_0603Metric"
 			(at 224.4852 66.04 0)
 			(effects
@@
 			)
 		)
-		(property "Footprint" "footprints:C_0402"
+		(property "Footprint" "footprints:C_0201_0603Metric"
 			(at 244.8052 66.04 0)
 			(effects
@@
 			)
 		)
-		(property "Footprint" "footprints:C_0402"
+		(property "Footprint" "footprints:C_0201_0603Metric"
 			(at 234.6452 66.04 0)
 			(effects
@@
 			)
 		)
-		(property "Value" "4.7nF"
+		(property "Value" "4.7uF"
 			(at 207.01 101.5999 0)
 			(effects
@@
 			)
 		)
-		(property "Footprint" "footprints:C_0402"
+		(property "Footprint" "footprints:C_0201_0603Metric"
 			(at 204.1652 85.09 0)
 			(effects

Commit message: ready for manufacturing
Parts:
- C34, C35: footprint footprints:C_0402 -> footprints:C_0201_0603Metric; LCSC PN c15195 -> c85930
- C36, C37, C38, C39, C40, C41, C42, C43, C44, C45, C46, C47, C48, C49, C50, C51: LCSC PN c307434 -> C88917
- C82, C83: LCSC PN C88915 -> C5383023
- C84: LCSC PN c84705 -> C2858031
- R96: footprint footprints:R_0402 -> footprints:R_0201_0603Metric; LCSC PN C105871 -> C138135
