File: HDMI.kicad_sch (KiCad schematic)
At the start: 50 parts, among them J10 10029449-001RLF, J11 10029449-001RLF, Q9 FDV301N, U11 NC7SZ125M5X, U24 TXS0102DCUR, U8 TXS0102DCUR

Commit message: new layout by abdul
Parts:
- removed R124, R131: 10K, footprints:R_0402, symbol Device:R_US
- removed U24, U8: TXS0102DCUR, footprints:SOP50P310X90-8N, symbol TXS0102DCUR:TXS0102DCUR
- added U2, U8: PCA9306TDCURQ1, footprints:DCU8, symbol PCA9306:PCA9306TDCURQ1
- C17, C22, C23, C24, C25: footprint footprints:C_0402 -> footprints:C_0201_0603Metric
Connections:
- net +3V3: now also U2.2 (VREF1), U8.2 (VREF1)
- net GNDREF: now also U2.1 (GND), U8.1 (GND)
- net HDMI_RX_SCL: now also U2.3 (SCL1)
- net HDMI_RX_SCL_LS: now also U2.6 (SCL2)
- net HDMI_RX_SDA: now also U2.4 (SDA1)
- net HDMI_RX_SDA_LS: now also U2.5 (SDA2)
- net HDMI_TX_SCL: now also U8.3 (SCL1)
- net HDMI_TX_SCL_LS: now also U8.6 (SCL2)
- net HDMI_TX_SDA: now also U8.4 (SDA1)
- net HDMI_TX_SDA_LS: now also U8.5 (SDA2)
- net at C17.1, R240.2: now also U8.7 (VREF2), U8.8 (EN)
- net at C24.1, R241.2: now also U2.7 (VREF2), U2.8 (EN)

Commit message: ready for manufacturing
Parts:
- C17, C22, C23, C24, C25: LCSC PN c1525 -> c307380
- J10, J11: LCSC PN C428493 -> (none)
- R154, R207: value 10K -> 10K 1%
- R155: footprint footprints:R_0402 -> footprints:R_0201_0603Metric; LCSC PN C105871 -> C138135
