File: HDMI.kicad_sch (KiCad schematic)
At the start: 48 parts, among them J10 10029449-001RLF, J11 10029449-001RLF, Q9 FDV301N, U11 NC7SZ125M5X, U2 PCA9306TDCURQ1, U8 PCA9306TDCURQ1

Commit message: post -production rework
Parts:
- removed C52: 1nF 250V, footprints:C_1808_4520Metric, symbol Device:C
- added C66: GA342DR7GF102KW02L, footprints:CAPC4520X220N, symbol GA342DR7GF102KW02L:GA342DR7GF102KW02L
Connections:
- net GNDREF: now also C66.1
- net VIDEO_SHIELD: now also C66.2
