File: PMOD,LED,SWITCHES.kicad_sch (KiCad schematic)
At the start: 71 parts, among them P1 PMOD-Device-x2-Type-Generic-A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, P2 PMOD-Device-x2-Type-Generic-A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, SW0 SW_SPDT, SW1 SW_SPDT, U27 TPD4E05U06DQAR, U28 TPD4E05U06DQAR, U29 TPD4E05U06DQAR, U30 TPD4E05U06DQAR, U31 MBT3904DW1T1G, U32 MBT3904DW1T1G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

Commit message: new layout by abdul
Parts:
- removed C7: 1uF / 10V, footprints:C_0402, symbol Device:C

Commit message: weekend update
Connections:
- net JA3_N: now also R75.1; no longer R76.1
- net JA3_P: now also R76.1; no longer R75.1
- net JA4_N: now also R77.1; no longer R78.1
- net JA4_P: now also R78.1; no longer R77.1
- net JB1_N: now also R71.1; no longer R72.1
- net JB1_P: now also R72.1; no longer R71.1
- net JB2_N: now also R73.1; no longer R74.1
- net JB2_P: now also R74.1; no longer R73.1
- net JB3_N: now also R79.1; no longer R80.1
- net JB3_P: now also R80.1; no longer R79.1
- net at P2.9 (P9), R77.2: now also U28.5 (D2-); no longer U28.4 (D2+)
- net at P2.10 (P10), R78.2: now also U28.4 (D2+); no longer U28.5 (D2-)
- net at P2.7 (P7), R75.2: now also U28.2 (D1-); no longer U28.1 (D1+)
- net at P2.8 (P8), R76.2: now also U28.1 (D1+); no longer U28.2 (D1-)
- net at P1.3 (P3), R73.2: now also U29.2 (D1-); no longer U29.1 (D1+)
- net at P1.4 (P4), R74.2: now also U29.1 (D1+); no longer U29.2 (D1-)
- net at P1.7 (P7), R79.2: now also U30.5 (D2-); no longer U30.4 (D2+)
- net at P1.8 (P8), R80.2: now also U30.4 (D2+); no longer U30.5 (D2-)

Commit message: ready for manufacturing
Parts:
- removed U30: TPD4E05U06DQAR, footprints:IC_TPD4E05U06DQAR, symbol TPD4E05U06DQAR:TPD4E05U06DQAR
- added H1: MH1, footprints:MountingHole_2.2mm_M2_Pad, symbol Mechanical:MountingHole_Pad
- added H2: MH2, footprints:MountingHole_2.2mm_M2_Pad, symbol Mechanical:MountingHole_Pad
- added H3: MH3, footprints:MountingHole_2.2mm_M2_Pad, symbol Mechanical:MountingHole_Pad
- added H4: MH4, footprints:MountingHole_2.2mm_M2_Pad, symbol Mechanical:MountingHole_Pad
- added U24: TPD4E05U06DQAR, footprints:IC_TPD4E05U06DQAR, symbol TPD4E05U06DQAR:TPD4E05U06DQAR
- C6: value 1uF /10V -> 1uF 10V; LCSC PN c14445 -> C52923
- D7, D8: LCSC PN C2909770 -> C20110230
- R15, R21, R22, R23, R24, R25, R26, R27, R28, R29: value 10k -> 10K 1%
- R30, R58: LCSC PN C295882 -> C830266
- R33, R34, R35, R55, R56, R57, R61, R62, R63, R64, R65, R66: value 2.2k -> 2.2K
- S6: value PTS645SK50SMTR92LFS -> BTN1; footprint footprints:SW_PTS645SK50SMTR92LFS -> footprints:TS-1002S-050xxC_XNP; LCSC PN C221872 -> C455110
- S7: value PTS645SK50SMTR92LFS -> BTN0; footprint footprints:SW_PTS645SK50SMTR92LFS -> footprints:TS-1002S-050xxC_XNP; LCSC PN C221872 -> C455110
- S8: value PTS645SK50SMTR92LFS -> BTN2; footprint footprints:SW_PTS645SK50SMTR92LFS -> footprints:TS-1002S-050xxC_XNP; LCSC PN C221872 -> C455110
- S9: value PTS645SK50SMTR92LFS -> BTN3; footprint footprints:SW_PTS645SK50SMTR92LFS -> footprints:TS-1002S-050xxC_XNP; LCSC PN C221872 -> C455110
Connections:
- net GND__1 is gone; now on net GNDREF: U27.8 (GND), U28.8 (GND)
- net GNDREF: now also U29.8 (GND), H1.1, H2.1, H3.1, H4.1, U24.3 (GND), U24.8 (GND)
- net at P2.1 (P1), R67.2: now also U24.1 (D1+); no longer U27.1 (D1+)
- net at P2.2 (P2), R68.2: now also U24.2 (D1-); no longer U27.2 (D1-)
- net at P2.3 (P3), R69.2: now also U24.4 (D2+); no longer U27.4 (D2+)
- net at P2.4 (P4), R70.2: now also U24.5 (D2-); no longer U27.5 (D2-)
- net at P1.1 (P1), R71.2: now also U27.5 (D2-); no longer U29.5 (D2-)
- net at P1.10 (P10), R82.2: now also U29.2 (D1-)
- net at P1.2 (P2), R72.2: now also U27.4 (D2+); no longer U29.4 (D2+)
- net at P1.3 (P3), R73.2: now also U27.2 (D1-); no longer U29.2 (D1-)
- net at P1.4 (P4), R74.2: now also U27.1 (D1+); no longer U29.1 (D1+)
- net at P1.7 (P7), R79.2: now also U29.5 (D2-)
- net at P1.8 (P8), R80.2: now also U29.4 (D2+)
- net at P1.9 (P9), R81.2: now also U29.1 (D1+)
