File: PMOD,LED,SWITCHES.kicad_sch (KiCad schematic)
At the start: 74 parts, among them P1 PMOD-Device-x2-Type-Generic-A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, P2 PMOD-Device-x2-Type-Generic-A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, SW0 SW_SPDT, SW1 SW_SPDT, U24 TPD4E05U06DQAR, U27 TPD4E05U06DQAR, U28 TPD4E05U06DQAR, U29 TPD4E05U06DQAR, U31 MBT3904DW1T1G, U32 MBT3904DW1T1G, U33 MBT3904DW1T1G

Commit message: post -production rework
Parts:
- D1, D4, D5, D6: LCSC PN C434449 -> C130723
Connections:
- net xJA4_N: now reaches P2.9 (P9), R77.2, U28.5 (D2-)
- net xJB4_P: now reaches P1.9 (P9), R81.2, U29.1 (D1+)
- net xJB4_N: now reaches P1.10 (P10), R82.2, U29.2 (D1-)
- net xJB3_P: now reaches P1.8 (P8), R80.2, U29.4 (D2+)
- net xJB3_N: now reaches P1.7 (P7), R79.2, U29.5 (D2-)
- net xJA1_P: now reaches P2.1 (P1), R67.2, U24.1 (D1+)
- net xJA1_N: now reaches P2.2 (P2), R68.2, U24.2 (D1-)
- net xJA2_P: now reaches P2.3 (P3), R69.2, U24.4 (D2+)
- net xJA2_N: now reaches P2.4 (P4), R70.2, U24.5 (D2-)
- net xJA4_P: now reaches P2.10 (P10), R78.2, U28.4 (D2+)
- net xJA3_N: now reaches P2.7 (P7), R75.2, U28.2 (D1-)
- net xJA3_P: now reaches P2.8 (P8), R76.2, U28.1 (D1+)
- net xJB1_N: now reaches P1.1 (P1), R71.2, U27.5 (D2-)
- net xJB1_P: now reaches P1.2 (P2), R72.2, U27.4 (D2+)
- net xJB2_N: now reaches P1.3 (P3), R73.2, U27.2 (D1-)
- net xJB2_P: now reaches P1.4 (P4), R74.2, U27.1 (D1+)
