File: SPDIF.kicad_sch (KiCad schematic)
At the start: 6 parts, among them U5 TOTX1950AF, U6 TORX1950AF

Commit message: ready for manufacturing
Parts:
- C10, C11: value .1uF -> 100nF 10V; LCSC PN c1525 -> C77020
- U5, U6: LCSC PN mouser -> (none)
Changed lines of the file:
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@@
 			)
 		)
-		(property "LCSC PN" "mouser"
+		(property "LCSC PN" ""
+			(at 128.27 58.42 0)
+			(effects
+				(font
+					(size 1.27 1.27)
+				)
+				(hide yes)
+			)
+		)
+		(property "Arrow Part Number" ""
+			(at 128.27 58.42 0)
+			(effects
+				(font
+					(size 1.27 1.27)
+				)
+				(hide yes)
+			)
+		)
+		(property "Arrow Price/Stock" ""
 			(at 128.27 58.42 0)
 			(effects
@@
 			)
 		)
-		(property "LCSC PN" "mouser"
+		(property "LCSC PN" ""
+			(at 133.35 110.49 0)
+			(effects
+				(font
+					(size 1.27 1.27)
+				)
+				(hide yes)
+			)
+		)
+		(property "Arrow Part Number" ""
+			(at 133.35 110.49 0)
+			(effects
+				(font
+					(size 1.27 1.27)
+				)
+				(hide yes)
+			)
+		)
+		(property "Arrow Price/Stock" ""
 			(at 133.35 110.49 0)
 			(effects
@@
 			)
 		)
-		(property "Value" ".1uF"
+		(property "Value" "100nF 10V"
 			(at 113.284 60.452 0)
 			(effects
@@
 			)
 		)
-		(property "LCSC PN" "c1525"
+		(property "LCSC PN" "C77020"
+			(at 119.38 60.96 0)
+			(effects
+				(font
+					(size 1.27 1.27)
+				)
+				(hide yes)
+			)
+		)
+		(property "Arrow Part Number" ""
+			(at 119.38 60.96 0)
+			(effects
+				(font
+					(size 1.27 1.27)
+				)
+				(hide yes)
+			)
+		)
+		(property "Arrow Price/Stock" ""
 			(at 119.38 60.96 0)
 			(effects
@@
 		(on_board yes)
 		(dnp no)
-		(fields_autoplaced yes)
 		(property "Reference" "C10"
-			(at 124.46 114.2999 0)
+			(at 121.666 113.03 0)
 			(effects
 				(font
@@
 			)
 		)
-		(property "Value" ".1uF"
-			(at 124.46 116.8399 0)
+		(property "Value" "100nF 10V"
+			(at 115.824 113.538 0)
 			(effects
 				(font
@@
 			)
 		)
-		(property "LCSC PN" "c1525"
+		(property "LCSC PN" "C77020"
+			(at 120.65 115.57 0)
+			(effects
+				(font
+					(size 1.27 1.27)
+				)
+				(hide yes)
+			)
+		)
+		(property "Arrow Part Number" ""
+			(at 120.65 115.57 0)
+			(effects
+				(font
+					(size 1.27 1.27)
+				)
+				(hide yes)
+			)
+		)
+		(property "Arrow Price/Stock" ""
 			(at 120.65 115.57 0)
 			(effects
@@
 		(on_board yes)
 		(dnp no)
-		(fields_autoplaced yes)
 		(property "Reference" "L1"
-			(at 127 114.3 90)
+			(at 127.508 120.65 90)
 			(effects
 				(font
@@
 		)
 		(property "Value" "47uH"
-			(at 127 116.84 90)
+			(at 127.762 119.126 90)
 			(effects
 				(font
@@
 		)
 		(property "LCSC PN" "C223186"
+			(at 127 119.38 0)
+			(effects
+				(font
+					(size 1.27 1.27)
+				)
+				(hide yes)
+			)
+		)
+		(property "Arrow Part Number" ""
+			(at 127 119.38 0)
+			(effects
+				(font
+					(size 1.27 1.27)
+				)
+				(hide yes)
+			)
+		)
+		(property "Arrow Price/Stock" ""
 			(at 127 119.38 0)
 			(effects
@@
 			(at 125.73 62.23 0)
 			(effects
+				(font
+					(size 1.27 1.27)
+				)
+				(hide yes)
+			)
+		)
+		(property "Arrow Part Number" ""
+			(at 125.73 62.23 0)
+			(effects
+				(font
+					(size 1.27 1.27)
+				)
+				(hide yes)
+			)
+		)
+		(property "Arrow Price/Stock" ""
+			(at 125.73 62.23 0)
+			(effects
