File: SPDIF.kicad_sch (KiCad schematic)
At the start: 6 parts, among them U5 TOTX1950AF, U6 TORX1950AF

Commit message: post -production rework
Parts:
- L1: LCSC PN C223186 -> C105499
Connections:
- net GNDREF: now also U6.5 (CASE), U6.6 (CASE)
