File: FPGA-BOARD.kicad_pcb (KiCad board)
At the start: 8 copper layers, 132.6 x 102.7 mm, 570 parts, among them IC1 IS43TR16256B-125KBLI, J1 PJ-102AH, J10 10029449-001RLF, J11 10029449-001RLF, J12 HFJ11-1G01ERL, J13 503398-1892, J14 PRT-14017, J15 USB-A-S-X-X-SM2, J16 10118194-0001LF, J17 Conn_01x02_Pin, J18 +3V3, J19 +1V8, J2 GND, J20 +1V5, J21 +1V0, J22 VCC_1V8IO, J3 Conn_01x03_Pin, J4 Conn_01x04_Pin, J5 Conn_01x02_Pin, J6 ADC_CONN, J7 JTAG Header, J8 Conn_01x02_Pin, J9 SJ1-3525NG, P1 PMOD-Device-x2-Type-Generic-A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, P2 PMOD-Device-x2-Type-Generic-A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, Q10 DMG2305UX-13, Q7 DMG2305UX-13, Q8 FDV301N, Q9 FDV301N, SW0 SW_SPDT, SW1 SW_SPDT, U1 XC7Z020-1CLG400I__, U10 TPD1E05U06DPYR, U11 NC7SZ125M5X, U12 RTL8211F-CG, U13 TXS02612RTWR, U14 TLV62130RGTT, U15 93LC56B-I/SN, U16 REF3012, U17 NC7WZ07P6X, U18 NL17SZ17XV5T2G, U19 NL17SZ17XV5T2G, U2 PCA9306TDCURQ1, U21 NC7WZ07P6X, U22 TPS65400RGZT, U23 NC7WZ07P6X, U24 TPD4E05U06DQAR, U25 TPS2051BDBVR, U26 TUSB1210BRHBT, U27 TPD4E05U06DQAR, U28 TPD4E05U06DQAR, U29 TPD4E05U06DQAR, U3 FT2232HQ, U30 TPD4E05U06DQAR, U31 MBT3904DW1T1G, U32 MBT3904DW1T1G, U33 MBT3904DW1T1G, U34 TPD1E05U06DPYR, U35 TPD1E05U06DPYR, U36 AD8592ARM, U37 TPD1E05U06DPYR, U38 TPD1E05U06DPYR, U39 TPD1E05U06DPYR, U4 ATSHA204A-SSHCZ-T, U40 TPS22918DBVR, U5 TOTX1950AF, U6 TORX1950AF, U7 S25FL128SAGMFI000, U8 PCA9306TDCURQ1, U9 SIP32510DT-T1-GE3, Y1 ABMM-25.000MHZ-B2-T, Y2 SG-8018CE_50.0000M-TJHPA, Y3 SIT1602AC-12-33E-12.000000G, Y4 ABM8G-26.000MHZ-18-D2Y-T

Commit message: post -production rework
Parts:
- removed C181: 1nF, footprints:C_0402
- removed D25: LED, footprints:LED_0402_1005Metric
- removed DONE1, led_rx1, led_tx1: Green, footprints:LED_0402_1005Metric
- removed J19: +1V8, footprints:PinHeader_1x01_P2.54mm_Vertical
- removed U7: S25FL128SAGMFI000, footprints:SO3016_INF
- added C222: GA342DR7GF102KW02L, footprints:CAPC4520X220N, B.Cu at (77.1, 102.3)
- added D10: LED, footprints:LED_0402_1005Metric, F.Cu at (96.9, 71.0)
- added D11: LED, footprints:LED_0402_1005Metric, F.Cu at (96.9, 69.9)
- added D3: LED, footprints:LED_0402_1005Metric, F.Cu at (109.6, 131.2)
- added D9: LED, footprints:LED_0402_1005Metric, F.Cu at (127.7, 94.2)
- added R216: 220, footprints:R_0402, F.Cu at (143.7, 81.6)
- added R217: 220, footprints:R_0402, F.Cu at (145.7, 81.7)
- added R219: 220, footprints:R_0402, F.Cu at (150.6, 81.6)
- added R220: 220, footprints:R_0402, B.Cu at (153.1, 82.3)
- added R221: 220, footprints:R_0402, F.Cu at (155.8, 81.6)
- added R222: 220, footprints:R_0402, F.Cu at (160.7, 81.6)
- added R223: 220, footprints:R_0402, F.Cu at (163.3, 81.6)
- added R224: 220, footprints:R_0402, F.Cu at (165.8, 81.6)
- added R225: 220, footprints:R_0402, F.Cu at (168.4, 81.6)
- added R226: 220, footprints:R_0402, F.Cu at (173.3, 74.6)
- added R227: 220, footprints:R_0402, F.Cu at (173.5, 81.6)
- added R228: 220, footprints:R_0402, F.Cu at (176.9, 81.7)
- added R229: 220, footprints:R_0402, F.Cu at (172.1, 81.6)
- added R230: 220, footprints:R_0402, F.Cu at (169.7, 81.6)
- added R231: 220, footprints:R_0402, F.Cu at (164.6, 81.7)
- added R232: 220, footprints:R_0402, F.Cu at (162.0, 81.6)
- added R233: 220, footprints:R_0402, F.Cu at (158.3, 81.6)
- added R242: 220, footprints:R_0402, F.Cu at (155.8, 74.1)
- added R243: 220, footprints:R_0402, F.Cu at (153.3, 74.1)
- added R244: 220, footprints:R_0402, B.Cu at (148.8, 82.4)
- added R245: 220, footprints:R_0402, B.Cu at (147.8, 82.4)
- added R246: 220, footprints:R_0402, F.Cu at (139.4, 81.6)
- added R247: 220, footprints:R_0402, F.Cu at (138.0, 73.9)
- added R248: 220, footprints:R_0402, B.Cu at (138.1, 82.2)
- added U20: NC7WZ07P6X, footprints:NC7WZ07P6X, F.Cu at (139.0, 123.0)
- C14, C184, C207, C9, R116, R38, R50, Y2: moved to F.Cu
- C172, C173, C174, C76, C77, U40, Y3: moved to B.Cu
- C52: value 1nF 250V -> GA342DR7GF102KW02L; footprint footprints:C_1808_4520Metric -> footprints:CAPC4520X220N; moved to B.Cu
- C66: value 1nF -> GA342DR7GF102KW02L; footprint footprints:C_0402 -> footprints:CAPC4520X220N; moved to F.Cu
- R189, R190, R192: value 2.2K -> 220
- R191: value 2.2K -> 220; moved to B.Cu
- U17: value NC7WZ07P6X -> W25Q128JVSIQ; footprint footprints:NC7WZ07P6X -> footprints:SOIC127P790X216-8N; moved to B.Cu
- moved J4 79.4 mm to (186.0, 127.8), turned to -90 degrees
- moved R46 78.9 mm to (184.4, 125.1)
- moved R48 73.2 mm to (182.8, 125.5), turned to 0 degrees
- moved R47 70.3 mm to (178.4, 124.5)
- moved R49 68.2 mm to (176.9, 125.0), turned to 0 degrees
- moved C66 67.3 mm to (129.4, 56.2), turned to -90 degrees
- moved C52 52.0 mm to (78.9, 68.5), turned to 0 degrees
- moved U17 37.7 mm to (170.6, 124.3)
- moved R94 36.6 mm to (107.8, 131.2), turned to 180 degrees
- moved R191 27.0 mm to (135.3, 73.5), turned to -90 degrees
- moved R192 21.5 mm to (139.9, 74.2), turned to 180 degrees
- moved J2 17.9 mm to (80.1, 143.5)
- moved R197 9.98 mm to (80.2, 86.9), turned to 180 degrees
- moved C14 9.60 mm to (168.6, 122.8)
- moved C173 6.48 mm to (134.5, 116.6), turned to 0 degrees
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Connections:
- net Net-(P1-P1) renamed /PMOD, LED, SWITCHES/xJB1_N
- net Net-(P1-P10) renamed /PMOD, LED, SWITCHES/xJB4_N
- net Net-(P1-P2) renamed /PMOD, LED, SWITCHES/xJB1_P
- net Net-(P1-P3) renamed /PMOD, LED, SWITCHES/xJB2_N
- net Net-(P1-P4) renamed /PMOD, LED, SWITCHES/xJB2_P
- net Net-(P1-P7) renamed /PMOD, LED, SWITCHES/xJB3_N
- net Net-(P1-P8) renamed /PMOD, LED, SWITCHES/xJB3_P
- net Net-(P1-P9) renamed /PMOD, LED, SWITCHES/xJB4_P
- net Net-(P2-P1) renamed /PMOD, LED, SWITCHES/xJA1_P
- net Net-(P2-P10) renamed /PMOD, LED, SWITCHES/xJA4_P
- net Net-(P2-P2) renamed /PMOD, LED, SWITCHES/xJA1_N
- net Net-(P2-P3) renamed /PMOD, LED, SWITCHES/xJA2_P
- net Net-(P2-P4) renamed /PMOD, LED, SWITCHES/xJA2_N
- net Net-(P2-P7) renamed /PMOD, LED, SWITCHES/xJA3_N
- net Net-(P2-P8) renamed /PMOD, LED, SWITCHES/xJA3_P
- net Net-(P2-P9) renamed /PMOD, LED, SWITCHES/xJA4_N
- C52 pad 1: VIDEO_SHIELD -> GNDREF
- C52 pad 2: GNDREF -> USB_SHIELD
- C66 pad 1: SHIELD -> GNDREF
- C66 pad 2: GNDREF -> VIDEO_SHIELD
- J12 pad 4: ETH_TD1_N -> ETH_TD2_P
- J12 pad 5: ETH_TD2_P -> ETH_TD2_N
- J12 pad 6: ETH_TD2_N -> ETH_TD1_N
- J14 pad 10: GPIO_15(UART_RX) -> Net-(J14-GPIO_15(UART_RX))
- J14 pad 11: GPIO_17 -> Net-(J14-GPIO_17)
- J14 pad 12: GPIO_18(PCM_CLK) -> Net-(J14-GPIO_18(PCM_CLK))
- J14 pad 13: GPIO_27 -> Net-(J14-GPIO_27)
- J14 pad 15: GPIO_22 -> Net-(J14-GPIO_22)
- J14 pad 16: GPIO_23 -> Net-(J14-GPIO_23)
- J14 pad 18: GPIO_24 -> Net-(J14-GPIO_24)
- J14 pad 19: GPIO_10(SPI_MOSI) -> Net-(J14-GPIO_10(SPIO_MOSI))
- J14 pad 21: GPIO_9(SPI_MISO) -> Net-(J14-GPIO_9(SPI0_MISO))
- J14 pad 22: GPIO_25 -> Net-(J14-GPIO_25)
- J14 pad 23: GPIO_11(SPI0_SCLK) -> Net-(J14-GPIO_11(SPI0_SCLK))
- J14 pad 24: GPIO_8(SPI0_CE0) -> Net-(J14-GPIO_8(SPI0_CE0))
- J14 pad 26: GPIO_7(SPI0_CE1) -> Net-(J14-GPIO_7(SPI0_CE1))
- J14 pad 27: GPIO_0(EEPROM_SDA) -> Net-(J14-GPIO_0(EEPROM_SDA))
- J14 pad 28: GPIO_1(EEPROM_SCL) -> Net-(J14-GPIO_1(EEPROM_SCL))
- J14 pad 29: GPIO_5 -> Net-(J14-GPIO_5)
- J14 pad 3: GPIO_2(I2C1_SDA) -> Net-(J14-GPIO2(I2C1_SDA))
- J14 pad 31: GPIO_6 -> Net-(J14-GPIO_6)
- J14 pad 32: GPIO_12(PWM0) -> Net-(J14-GPIO_12(PWM0))
- J14 pad 33: GPIO_13(PWM1) -> Net-(J14-GPIO_13(PWM1))
- J14 pad 35: GPIO_19(PCM_FS) -> Net-(J14-GPIO_19(PCM_FS))
- J14 pad 36: GPIO_16 -> Net-(J14-GPIO_16)
- J14 pad 37: GPIO_26 -> Net-(J14-GPIO_26)
- J14 pad 38: GPIO_20(PCM_DIN) -> Net-(J14-GPIO_20(PCM_DIN))
- J14 pad 40: GPIO_21(PCM_DOUT) -> Net-(J14-GPIO_21(PCM_DOUT))
- J14 pad 5: GPIO_3(I2C1_SCL) -> Net-(J14-GPIO_3(I2C1_SCL))
- J14 pad 7: GPIO_4(GPCLK0) -> Net-(J14-GPIO_4(GPCLK0))
- J14 pad 8: GPIO_14(UART_TX) -> Net-(J14-GPIO_14(UART_TX))
- J8 pad 2: unconnected-(J8-Pin_2-Pad2) -> +3V3
- J9 pad 2: Net-(J9-Pad2) -> Net-(F2-Pad2)
- J9 pad 3: Net-(F2-Pad2) -> Net-(J9-Pad3)
- R111 pad 2: UART_TXD -> UART_RXD_OUT
- R112 pad 1: Net-(U3-ADBUS5) -> Net-(U3-ADBUS6)
- R189 pad 2: +3V3 -> Net-(J14-GPIO2(I2C1_SDA))
- R190 pad 2: +3V3 -> Net-(J14-GPIO_3(I2C1_SCL))
- R191 pad 1: GPIO_0(EEPROM_SDA) -> GPIO_4(GPCLK0)
- R191 pad 2: +3V3 -> Net-(J14-GPIO_4(GPCLK0))
- R192 pad 1: GPIO_1(EEPROM_SCL) -> GPIO_17
- R192 pad 2: +3V3 -> Net-(J14-GPIO_17)
- R197 pad 1: Net-(J9-Pad2) -> Net-(J9-Pad3)
- R51 pad 2: UART_RXD -> UART_TXD_IN
- U1 pad C5: UART_TXD -> UART_TXD_IN
- U1 pad C8: UART_RXD -> UART_RXD_OUT
- U13 pad V: GNDREF -> (no net)
- U14 pad 18: GNDREF -> (no net)
- U14 pad 19: GNDREF -> (no net)
- U14 pad 20: GNDREF -> (no net)
- U14 pad 21: GNDREF -> (no net)
- U14 pad 22: GNDREF -> (no net)
- U17 pad 1: VCC1V8_IO_EDGE -> SPI_CS
- U17 pad 2: GNDREF -> SPI_DQ1/MODE1
- U17 pad 3: unconnected-(U17A-A2-Pad3) -> SPI_DQ2/MODE2
- U17 pad 4: unconnected-(U17A-Y2-Pad4) -> GNDREF
- U17 pad 5: +1V8 -> SPI_DQ0/MODE3
- U17 pad 6: ETH_RST_B -> SPI_SCK/MODE4
- U22 pad V: GNDREF -> (no net)
- U26 pad V: GNDREF -> (no net)
- U3 pad 21: unconnected-(U3-ADBUS4-Pad21) -> +3V3
- U3 pad 22: Net-(U3-ADBUS5) -> unconnected-(U3-ADBUS5-Pad22)
- U3 pad 23: unconnected-(U3-ADBUS6-Pad23) -> Net-(U3-ADBUS6)
- U30 pad 10: GNDREF -> (no net)
- U6 pad 5: unconnected-(U6-CASE-Pad5) -> GNDREF
- U6 pad 6: unconnected-(U6-CASE-Pad6) -> GNDREF
Routing:
- net SPI_DQ2/MODE2: track 174.7 -> 40.7 mm, vias 3 -> 1
- net SPI_DQ3/MODE0: track 162.5 -> 41.6 mm, vias 3 -> 1
- net UART_TXD: track 88.9 -> 0.00 mm, vias 2 -> 0
- net UART_TXD_IN: track 0.00 -> 87.5 mm, vias 0 -> 2
- net UART_RXD_OUT: track 0.00 -> 84.0 mm, vias 0 -> 2
- net UART_RXD: track 82.7 -> 0.00 mm, vias 2 -> 0
- net Net-(Q8-Pad3): track 2.53 -> 45.1 mm
- net USBHOST_DATA7: track 100.6 -> 75.8 mm
- net USBHOST_DATA4: track 99.3 -> 75.0 mm
- net USBHOST_DATA6: track 101.3 -> 78.0 mm
- net USBHOST_DATA1: track 99.3 -> 76.5 mm
- net USBHOST_DATA3: track 98.4 -> 79.0 mm
- net USBHOST_NXT: track 95.1 -> 76.3 mm
- net GNDREF: track 259.3 -> 278.1 mm, vias 579 -> 653
- net USBHOST_DATA0: track 101.4 -> 83.3 mm
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Other:
- board size 132.6 x 102.7 mm -> 132.6 x 97.9 mm
- board text added: "100Mb"
- board text added: "10Mb"
- board text added: "1Gb"
- board text added: "Designed By ABDUL AJADI"
- board text added: "PORB"
- board text removed: "+1V8"
- board text removed: "BY ABDUL AJADI"
- board text removed: "JTAG"
- board text removed: "PROTO 1"
- board text removed: "QSPI"
- board text removed: "SD"
