File: FPGA-BOARD.kicad_pcb (KiCad board)
At the start: 8 copper layers, 132.6 x 97.9 mm, 593 parts, among them IC1 IS43TR16256B-125KBLI, J1 PJ-102AH, J10 10029449-001RLF, J11 10029449-001RLF, J12 HFJ11-1G01ERL, J13 503398-1892, J14 PRT-14017, J15 USB-A-S-X-X-SM2, J16 10118194-0001LF, J17 Conn_01x02_Pin, J18 +3V3, J2 GND, J20 +1V5, J21 +1V0, J22 VCC_1V8IO, J3 Conn_01x03_Pin, J4 Conn_01x04_Pin, J5 Conn_01x02_Pin, J6 ADC_CONN, J7 JTAG Header, J8 Conn_01x02_Pin, J9 SJ1-3525NG, P1 PMOD-Device-x2-Type-Generic-A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, P2 PMOD-Device-x2-Type-Generic-A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, Q10 DMG2305UX-13, Q7 DMG2305UX-13, Q8 FDV301N, Q9 FDV301N, SW0 SW_SPDT, SW1 SW_SPDT, U1 XC7Z020-1CLG400I__, U10 TPD1E05U06DPYR, U11 NC7SZ125M5X, U12 RTL8211F-CG, U13 TXS02612RTWR, U14 TLV62130RGTT, U15 93LC56B-I/SN, U16 REF3012, U17 W25Q128JVSIQ, U18 NL17SZ17XV5T2G, U19 NL17SZ17XV5T2G, U2 PCA9306TDCURQ1, U20 NC7WZ07P6X, U21 NC7WZ07P6X, U22 TPS65400RGZT, U23 NC7WZ07P6X, U24 TPD4E05U06DQAR, U25 TPS2051BDBVR, U26 TUSB1210BRHBT, U27 TPD4E05U06DQAR, U28 TPD4E05U06DQAR, U29 TPD4E05U06DQAR, U3 FT2232HQ, U30 TPD4E05U06DQAR, U31 MBT3904DW1T1G, U32 MBT3904DW1T1G, U33 MBT3904DW1T1G, U34 TPD1E05U06DPYR, U35 TPD1E05U06DPYR, U36 AD8592ARM, U37 TPD1E05U06DPYR, U38 TPD1E05U06DPYR, U39 TPD1E05U06DPYR, U4 ATSHA204A-SSHCZ-T, U40 TPS22918DBVR, U5 TOTX1950AF, U6 TORX1950AF, U8 PCA9306TDCURQ1, U9 SIP32510DT-T1-GE3, Y1 ABMM-25.000MHZ-B2-T, Y2 SG-8018CE_50.0000M-TJHPA, Y3 SIT1602AC-12-33E-12.000000G, Y4 ABM8G-26.000MHZ-18-D2Y-T

Commit message: KICAD 10 DRC fixes
Connections:
- U13 pad V: (no net) -> GNDREF
- U14 pad 18: (no net) -> GNDREF
- U14 pad 19: (no net) -> GNDREF
- U14 pad 20: (no net) -> GNDREF
- U14 pad 21: (no net) -> GNDREF
- U14 pad 22: (no net) -> GNDREF
- U22 pad V: (no net) -> GNDREF
- U26 pad V: (no net) -> GNDREF
Routing:
- net GNDREF: track 278.1 -> 280.8 mm
